File: power.kicad_sch (KiCad schematic)
At the start: 1 part, among them U40 RP2040

Commit message: Before 10K resistors change
Parts:
- added C69, C70, C71, C72, C73, C74: C, symbol Device:C
- added J1: USB_C_Receptacle_USB2.0_16P, symbol Connector:USB_C_Receptacle_USB2.0_16P
- added R48, R49, R50: R, symbol Device:R
- added U41: W25Q128JVS, Package_SO:SOIC-8_5.3x5.3mm_P1.27mm, symbol Memory_Flash:W25Q128JVS
- added U42: MIC5219-3.3YM5, Package_TO_SOT_SMD:SOT-23-5, symbol Regulator_Linear:MIC5219-3.3YM5
- added Y1: 12MHz, symbol Device:Crystal
Connections:
- net GND: now also C69.1, C70.1, C71.1, C72.1, C73.1, C74.1, J1.A1 (GND), J1.A12 (GND), J1.B1 (GND), J1.B12 (GND), J1.S1 (SHIELD), R48.2, R49.2, U41.4 (GND), U42.2 (GND)
- net VCC: now reaches U40.1 (IOVDD), U40.10 (IOVDD), U40.22 (IOVDD), U40.33 (IOVDD), U40.42 (IOVDD), U40.49 (IOVDD)
- net VCC: now also U40.43 (ADC_AVDD), U40.44 (VREG_IN), U40.48 (USB_VDD), C71.2, C72.2, C73.2, C74.2, R50.2, U42.5 (OUT)
- net at U40.23 (DVDD), U40.50 (DVDD): now also U40.45 (VREG_VOUT), C69.2
- net at U40.26 (RUN): now also R50.1
- net data_n: now reaches U40.46 (USB_DM)
- net data_n: now also J1.A7 (D-), J1.B7 (D-)
- net data_p: now reaches U40.47 (USB_DP)
- net data_p: now also J1.A6 (D+), J1.B6 (D+)
- net at U40.51 (QSPI_SD3): now also U41.7 (~{HOLD}/~{RESET}/IO_{3})
- net at U40.52 (QSPI_SCLK): now also U41.6 (CLK)
- net at U40.53 (QSPI_SD0): now also U41.5 (DI/IO_{0})
- net at U40.54 (QSPI_SD2): now also U41.3 (~{WP}/IO_{2})
- net at U40.55 (QSPI_SD1): now also U41.2 (DO/IO_{1})
- net at U40.56 (QSPI_SS): now also U41.1 (~{CS})
- new net: C70.2, U41.8 (VCC)
- new net: J1.A5 (CC1), R48.1
- new net: J1.A4 (VBUS), J1.A9 (VBUS), J1.B4 (VBUS), J1.B9 (VBUS), U42.1 (IN)
- new net: J1.B5 (CC2), R49.1
Other:
- moved on the sheet: U40

Commit message: Before capcitor update
Parts:
- R48, R49: value R -> 5.1k
Changed lines of the file:
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@@
 		(dnp no)
 		(property "Reference" "R48"
-			(at 93.472 70.358 90)
-			(effects
-				(font
-					(size 1.27 1.27)
-				)
-			)
-		)
-		(property "Value" "R"
+			(at 94.996 70.358 90)
+			(effects
+				(font
+					(size 1.27 1.27)
+				)
+			)
+		)
+		(property "Value" "5.1k"
 			(at 90.678 70.358 90)
 			(effects
@@
 		(dnp no)
 		(property "Reference" "R49"
-			(at 93.726 77.47 90)
-			(effects
-				(font
-					(size 1.27 1.27)
-				)
-			)
-		)
-		(property "Value" "R"
+			(at 94.742 77.47 90)
+			(effects
+				(font
+					(size 1.27 1.27)
+				)
+			)
+		)
+		(property "Value" "5.1k"
 			(at 90.678 77.47 90)
 			(effects

Commit message: updated capacitor values
Parts:
- C69, C70, C71, C72, C73, C74: value C -> 100nF
Changed lines of the file:
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@@
 			)
 		)
-		(property "Value" "C"
+		(property "Value" "100nF"
 			(at 144.78 59.6899 0)
 			(effects
@@
 			)
 		)
-		(property "Value" "C"
+		(property "Value" "100nF"
 			(at 184.658 34.798 0)
 			(effects
@@
 			)
 		)
-		(property "Value" "C"
+		(property "Value" "100nF"
 			(at 215.392 21.082 90)
 			(effects
@@
 			)
 		)
-		(property "Value" "C"
+		(property "Value" "100nF"
 			(at 215.392 33.782 90)
 			(effects
@@
 			)
 		)
-		(property "Value" "C"
+		(property "Value" "100nF"
 			(at 215.392 27.432 90)
 			(effects
@@
 			)
 		)
-		(property "Value" "C"
+		(property "Value" "100nF"
 			(at 215.392 40.132 90)
 			(effects

Commit message: Updated: power
Parts:
- added C75, C76: 15pF, symbol Device:C
- added C77: 470pF, symbol Device:C
- added C78, C79: 10µF, symbol Device:C
- added C80: 1µF, symbol Device:C
- added R51: 1k, Resistor_SMD:R_1206_3216Metric_Pad1.30x1.75mm_HandSolder, symbol Device:R
- C69: value 100nF -> 1µF
- R48, R49: footprint (none) -> Resistor_SMD:R_1206_3216Metric_Pad1.30x1.75mm_HandSolder
- R50: value R -> 10k; footprint (none) -> Resistor_SMD:R_1206_3216Metric_Pad1.30x1.75mm_HandSolder
Connections:
- net GND: now also C75.2, C76.2, C77.2, C78.2, C79.2, C80.2
- net VCC: now also C70.2, U41.8 (VCC), C79.1
- net at J1.A4 (VBUS), J1.A9 (VBUS), J1.B4 (VBUS)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: now also U42.3 (EN), C78.1, C80.1
- net at U40.20 (XIN): now also Y1.1, C76.1
- net at U40.21 (XOUT): now also R51.2
- net SRCLK: now reaches U40.4 (GPIO2)
- net ser: now reaches U40.5 (GPIO3)
- net RCLK: now reaches U40.6 (GPIO4)
- net at U42.4 (BP): now also C77.1
- net at Y1.2: now also C75.1, R51.1
Other:
- moved on the sheet: C69, C70, C71, C72, C73, C74, J1, R48, R49, R50, U40, U41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

Commit message: Updated: op amps
Parts:
- C69, C70, C71, C72, C73, C74, C75, C76, C77, C78, C79, C80: footprint (none) -> Capacitor_SMD:C_1206_3216Metric_Pad1.33x1.80mm_HandSolder
Connections:
- net CLK: now reaches U40.13 (GPIO10)
- net SDI: now reaches U40.14 (GPIO11)
Changed lines of the file:
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@@
+		)
+	)
+	(global_label "CLK"
+		(shape output)
+		(at 219.71 88.9 0)
+		(fields_autoplaced yes)
+		(effects
+			(font
+				(size 1.27 1.27)
+			)
+			(justify left)
+		)
+		(property "Intersheetrefs" "${INTERSHEET_REFS}"
+			(at 226.2633 88.9 0)
+			(effects
+				(font
+					(size 1.27 1.27)
+				)
+				(justify left)
+				(hide yes)
+			)
 		)
 	)
@@
 		)
 	)
+	(global_label "SDI"
+		(shape output)
+		(at 219.71 91.44 0)
+		(fields_autoplaced yes)
+		(effects
+			(font
+				(size 1.27 1.27)
+			)
+			(justify left)
+		)
+		(property "Intersheetrefs" "${INTERSHEET_REFS}"
+			(at 225.7795 91.44 0)
+			(effects
+				(font
+					(size 1.27 1.27)
+				)
+				(justify left)
+				(hide yes)
+			)
+		)
+	)
 	(global_label "VCC"
 		(shape input)
@@
 			)
 		)
-		(property "Footprint" ""
+		(property "Footprint" "Capacitor_SMD:C_1206_3216Metric_Pad1.33x1.80mm_HandSolder"
 			(at 149.5552 68.58 0)
 			(effects
@@
 			)
 		)
-		(property "Footprint" ""
+		(property "Footprint" "Capacitor_SMD:C_1206_3216Metric_Pad1.33x1.80mm_HandSolder"
 			(at 147.32 122.8852 0)
 			(effects
@@
 			)
 		)
-		(property "Footprint" ""
+		(property "Footprint" "Capacitor_SMD:C_1206_3216Metric_Pad1.33x1.80mm_HandSolder"
 			(at 79.7052 64.77 0)
 			(effects
@@
 			)
 		)
-		(property "Footprint" ""
+		(property "Footprint" "Capacitor_SMD:C_1206_3216Metric_Pad1.33x1.80mm_HandSolder"
 			(at 101.2952 62.23 0)
 			(effects
@@
 			)
 		)
-		(property "Footprint" ""
+		(property "Footprint" "Capacitor_SMD:C_1206_3216Metric_Pad1.33x1.80mm_HandSolder"
 			(at 190.1952 52.07 0)
 			(effects
@@
 			)
 		)
-		(property "Footprint" ""
+		(property "Footprint" "Capacitor_SMD:C_1206_3216Metric_Pad1.33x1.80mm_HandSolder"
 			(at 104.14 47.2948 0)
 			(effects
@@
 			)
 		)
-		(property "Footprint" ""
+		(property "Footprint" "Capacitor_SMD:C_1206_3216Metric_Pad1.33x1.80mm_HandSolder"
 			(at 217.17 33.9852 0)
 			(effects
@@
 			)
 		)
-		(property "Footprint" ""
+		(property "Footprint" "Capacitor_SMD:C_1206_3216Metric_Pad1.33x1.80mm_HandSolder"
 			(at 67.6148 41.91 0)
 			(effects
@@
 			)
 		)
-		(property "Footprint" ""
+		(property "Footprint" "Capacitor_SMD:C_1206_3216Metric_Pad1.33x1.80mm_HandSolder"
 			(at 147.32 112.7252 0)
 			(effects
@@
 			)
 		)
-		(property "Footprint" ""
+		(property "Footprint" "Capacitor_SMD:C_1206_3216Metric_Pad1.33x1.80mm_HandSolder"
 			(at 217.17 46.6852 0)
 			(effects
@@
 			)
 		)
-		(property "Footprint" ""
+		(property "Footprint" "Capacitor_SMD:C_1206_3216Metric_Pad1.33x1.80mm_HandSolder"
 			(at 217.17 40.3352 0)
 			(effects
@@
 			)
 		)
-		(property "Footprint" ""
+		(property "Footprint" "Capacitor_SMD:C_1206_3216Metric_Pad1.33x1.80mm_HandSolder"
 			(at 217.17 53.0352 0)
 			(effects

Commit message: Updated: pots
Parts:
- added C81: 10µF, symbol Device:C
- added C82: 100nF, symbol Device:C
- added R52, R53: 10k, symbol Device:R
- added U2: TLV9061xDBV, Package_TO_SOT_SMD:SOT-23-5, symbol Amplifier_Operational:TLV9061xDBV
Connections:
- net GND: now also C81.1, C82.1, R53.2, U2.2 (V-)
- net VCC: now also R52.1, U2.5 (V+)
- new net: C82.2, R52.2, R53.1, U2.3 (+)
- new net VREF: C81.2, U2.1, U2.4 (-)
Other:
- moved on the sheet: C77, C78, C79, C80, J1, R48, R49, U42
