File: analog_NN.kicad_pcb (KiCad board)
At the start: 2 copper layers, 64 parts, among them U28 AD5160, U29 AD5160, U30 AD5160, U31 AD5160, U32 AD5160, U33 AD5160, U34 AD5160, U35 AD5160, U36 AD5160, U37 AD5160, U38 AD5160, U39 AD5160, U40 AD5160, U41 AD5160, U42 AD5160, U43 AD5160, U44 AD5160, U45 AD5160, U46 AD5160, U47 AD5160, U48 AD5160, U49 AD5160, U50 AD5160, U51 AD5160, U52 AD5160, U53 AD5160, U54 AD5160, U55 AD5160, U56 AD5160, U57 AD5160, U58 AD5160, U59 AD5160, U60 AD5160, U61 AD5160, U62 AD5160, U63 AD5160, U64 AD5160, U65 AD5160, U66 AD5160, U67 AD5160, U68 AD5160, U69 AD5160, U70 AD5160, U71 AD5160, U72 AD5160, U73 AD5160, U74 AD5160, U75 AD5160, U76 AD5160, U77 AD5160, U78 AD5160, U79 AD5160, U80 AD5160, U81 AD5160, U82 AD5160, U83 AD5160, U84 AD5160, U85 AD5160, U86 AD5160, U87 AD5160, U88 AD5160, U89 AD5160, U90 AD5160, U91 AD5160

Commit message: Updated: crossbar
Parts:
- removed U44, U45, U46, U47, U48, U49, U50, U51, U52, U53, U54, U55, U56, U57, U58, U59, U84, U85, U86, U87, U88, U89, U90, U91: AD5160, Package_TO_SOT_SMD:SOT-23-8
- added C1: 100nF, Capacitor_SMD:C_1206_3216Metric_Pad1.33x1.80mm_HandSolder, F.Cu at (66.6, 114.3)
- added C10: 100nF, Capacitor_SMD:C_1206_3216Metric_Pad1.33x1.80mm_HandSolder, F.Cu at (93.8, 111.2)
- added C11: 100nF, Capacitor_SMD:C_1206_3216Metric_Pad1.33x1.80mm_HandSolder, F.Cu at (99.8, 94.5)
- added C12: 100nF, Capacitor_SMD:C_1206_3216Metric_Pad1.33x1.80mm_HandSolder, F.Cu at (99.8, 97.8)
- added C13: 100nF, Capacitor_SMD:C_1206_3216Metric_Pad1.33x1.80mm_HandSolder, F.Cu at (99.8, 101.2)
- added C14: 100nF, Capacitor_SMD:C_1206_3216Metric_Pad1.33x1.80mm_HandSolder, F.Cu at (99.8, 104.5)
- added C15: 100nF, Capacitor_SMD:C_1206_3216Metric_Pad1.33x1.80mm_HandSolder, F.Cu at (99.8, 107.9)
- added C16: 100nF, Capacitor_SMD:C_1206_3216Metric_Pad1.33x1.80mm_HandSolder, F.Cu at (99.8, 111.2)
- added C17: 100nF, Capacitor_SMD:C_1206_3216Metric_Pad1.33x1.80mm_HandSolder, F.Cu at (105.8, 94.5)
- added C18: 100nF, Capacitor_SMD:C_1206_3216Metric_Pad1.33x1.80mm_HandSolder, F.Cu at (105.8, 97.8)
- added C19: 100nF, Capacitor_SMD:C_1206_3216Metric_Pad1.33x1.80mm_HandSolder, F.Cu at (105.8, 101.2)
- added C2: 100nF, Capacitor_SMD:C_1206_3216Metric_Pad1.33x1.80mm_HandSolder, F.Cu at (66.6, 117.7)
- added C20: 100nF, Capacitor_SMD:C_1206_3216Metric_Pad1.33x1.80mm_HandSolder, F.Cu at (105.8, 104.5)
- added C21: 100nF, Capacitor_SMD:C_1206_3216Metric_Pad1.33x1.80mm_HandSolder, F.Cu at (105.8, 107.9)
- added C22: 100nF, Capacitor_SMD:C_1206_3216Metric_Pad1.33x1.80mm_HandSolder, F.Cu at (105.8, 111.2)
- added C23: 100nF, Capacitor_SMD:C_1206_3216Metric_Pad1.33x1.80mm_HandSolder, F.Cu at (111.8, 94.5)
- added C24: 100nF, Capacitor_SMD:C_1206_3216Metric_Pad1.33x1.80mm_HandSolder, F.Cu at (111.8, 97.8)
- added C25: 100nF, Capacitor_SMD:C_1206_3216Metric_Pad1.33x1.80mm_HandSolder, F.Cu at (111.8, 101.2)
- added C26: 100nF, Capacitor_SMD:C_1206_3216Metric_Pad1.33x1.80mm_HandSolder, F.Cu at (111.8, 104.5)
- added C27: 100nF, Capacitor_SMD:C_1206_3216Metric_Pad1.33x1.80mm_HandSolder, F.Cu at (111.8, 107.9)
- added C28: 100nF, Capacitor_SMD:C_1206_3216Metric_Pad1.33x1.80mm_HandSolder, F.Cu at (111.8, 111.2)
- added C29: 100nF, Capacitor_SMD:C_1206_3216Metric_Pad1.33x1.80mm_HandSolder, F.Cu at (71.8, 60.3)
- added C3: 100nF, Capacitor_SMD:C_1206_3216Metric_Pad1.33x1.80mm_HandSolder, F.Cu at (66.6, 121.0)
- added C30: 100nF, Capacitor_SMD:C_1206_3216Metric_Pad1.33x1.80mm_HandSolder, F.Cu at (71.8, 63.6)
- added C31: 100nF, Capacitor_SMD:C_1206_3216Metric_Pad1.33x1.80mm_HandSolder, F.Cu at (71.8, 67.0)
- added C32: 100nF, Capacitor_SMD:C_1206_3216Metric_Pad1.33x1.80mm_HandSolder, F.Cu at (71.8, 70.3)
- added C33: 100nF, Capacitor_SMD:C_1206_3216Metric_Pad1.33x1.80mm_HandSolder, F.Cu at (71.8, 73.7)
- added C34: 100nF, Capacitor_SMD:C_1206_3216Metric_Pad1.33x1.80mm_HandSolder, F.Cu at (71.8, 77.0)
- added C35: 100nF, Capacitor_SMD:C_1206_3216Metric_Pad1.33x1.80mm_HandSolder, F.Cu at (71.8, 80.4)
- added C36: 100nF, Capacitor_SMD:C_1206_3216Metric_Pad1.33x1.80mm_HandSolder, F.Cu at (71.8, 83.7)
- added C37: 100nF, Capacitor_SMD:C_1206_3216Metric_Pad1.33x1.80mm_HandSolder, F.Cu at (71.8, 87.1)
- added C38: 100nF, Capacitor_SMD:C_1206_3216Metric_Pad1.33x1.80mm_HandSolder, F.Cu at (77.8, 60.3)
- added C39: 100nF, Capacitor_SMD:C_1206_3216Metric_Pad1.33x1.80mm_HandSolder, F.Cu at (77.8, 63.6)
- added C4: 100nF, Capacitor_SMD:C_1206_3216Metric_Pad1.33x1.80mm_HandSolder, F.Cu at (66.6, 124.4)
- added C40: 100nF, Capacitor_SMD:C_1206_3216Metric_Pad1.33x1.80mm_HandSolder, F.Cu at (77.8, 67.0)
- added C41: 100nF, Capacitor_SMD:C_1206_3216Metric_Pad1.33x1.80mm_HandSolder, F.Cu at (77.8, 70.3)
- added C42: 100nF, Capacitor_SMD:C_1206_3216Metric_Pad1.33x1.80mm_HandSolder, F.Cu at (77.8, 73.7)
- added C43: 100nF, Capacitor_SMD:C_1206_3216Metric_Pad1.33x1.80mm_HandSolder, F.Cu at (77.8, 77.0)
- added C44: 100nF, Capacitor_SMD:C_1206_3216Metric_Pad1.33x1.80mm_HandSolder, F.Cu at (77.8, 80.4)
- added C45: 100nF, Capacitor_SMD:C_1206_3216Metric_Pad1.33x1.80mm_HandSolder, F.Cu at (77.8, 83.7)
- added C46: 100nF, Capacitor_SMD:C_1206_3216Metric_Pad1.33x1.80mm_HandSolder, F.Cu at (77.8, 87.1)
- added C47: 100nF, Capacitor_SMD:C_1206_3216Metric_Pad1.33x1.80mm_HandSolder, F.Cu at (83.8, 60.3)
- added C48: 100nF, Capacitor_SMD:C_1206_3216Metric_Pad1.33x1.80mm_HandSolder, F.Cu at (83.8, 63.6)
- added C49: 100nF, Capacitor_SMD:C_1206_3216Metric_Pad1.33x1.80mm_HandSolder, F.Cu at (83.8, 67.0)
- added C5: 100nF, Capacitor_SMD:C_1206_3216Metric_Pad1.33x1.80mm_HandSolder, F.Cu at (93.8, 94.5)
- added C50: 100nF, Capacitor_SMD:C_1206_3216Metric_Pad1.33x1.80mm_HandSolder, F.Cu at (83.8, 70.3)
- added C51: 100nF, Capacitor_SMD:C_1206_3216Metric_Pad1.33x1.80mm_HandSolder, F.Cu at (83.8, 73.7)
- added C52: 100nF, Capacitor_SMD:C_1206_3216Metric_Pad1.33x1.80mm_HandSolder, F.Cu at (83.8, 77.0)
- added C53: 100nF, Capacitor_SMD:C_1206_3216Metric_Pad1.33x1.80mm_HandSolder, F.Cu at (83.8, 80.4)
- added C54: 100nF, Capacitor_SMD:C_1206_3216Metric_Pad1.33x1.80mm_HandSolder, F.Cu at (83.8, 83.7)
- added C55: 100nF, Capacitor_SMD:C_1206_3216Metric_Pad1.33x1.80mm_HandSolder, F.Cu at (83.8, 87.1)
- added C56: 100nF, Capacitor_SMD:C_1206_3216Metric_Pad1.33x1.80mm_HandSolder, F.Cu at (89.8, 60.3)
- added C57: 100nF, Capacitor_SMD:C_1206_3216Metric_Pad1.33x1.80mm_HandSolder, F.Cu at (89.8, 63.6)
- added C58: 100nF, Capacitor_SMD:C_1206_3216Metric_Pad1.33x1.80mm_HandSolder, F.Cu at (89.8, 67.0)
- added C59: 100nF, Capacitor_SMD:C_1206_3216Metric_Pad1.33x1.80mm_HandSolder, F.Cu at (89.8, 70.3)
- added C6: 100nF, Capacitor_SMD:C_1206_3216Metric_Pad1.33x1.80mm_HandSolder, F.Cu at (93.8, 97.8)
- added C60: 100nF, Capacitor_SMD:C_1206_3216Metric_Pad1.33x1.80mm_HandSolder, F.Cu at (89.8, 73.7)
- added C61: 100nF, Capacitor_SMD:C_1206_3216Metric_Pad1.33x1.80mm_HandSolder, F.Cu at (80.6, 94.5)
- added C62: 100nF, Capacitor_SMD:C_1206_3216Metric_Pad1.33x1.80mm_HandSolder, F.Cu at (80.6, 97.8)
- added C63: 100nF, Capacitor_SMD:C_1206_3216Metric_Pad1.33x1.80mm_HandSolder, F.Cu at (80.6, 101.2)
- added C64: 100nF, Capacitor_SMD:C_1206_3216Metric_Pad1.33x1.80mm_HandSolder, F.Cu at (80.6, 104.5)
- added C65: 100nF, Capacitor_SMD:C_1206_3216Metric_Pad1.33x1.80mm_HandSolder, F.Cu at (80.6, 107.9)
- added C66: 100nF, Capacitor_SMD:C_1206_3216Metric_Pad1.33x1.80mm_HandSolder, F.Cu at (80.6, 111.2)
- added C67: 100nF, Capacitor_SMD:C_1206_3216Metric_Pad1.33x1.80mm_HandSolder, F.Cu at (80.6, 114.6)
- added C68: 100nF, Capacitor_SMD:C_1206_3216Metric_Pad1.33x1.80mm_HandSolder, F.Cu at (80.6, 117.9)
- added C69: 1µF, Capacitor_SMD:C_1206_3216Metric_Pad1.33x1.80mm_HandSolder, F.Cu at (93.8, 116.6)
- added C7: 100nF, Capacitor_SMD:C_1206_3216Metric_Pad1.33x1.80mm_HandSolder, F.Cu at (93.8, 101.2)
- added C70: 100nF, Capacitor_SMD:C_1206_3216Metric_Pad1.33x1.80mm_HandSolder, F.Cu at (93.8, 119.9)
- added C71: 100nF, Capacitor_SMD:C_1206_3216Metric_Pad1.33x1.80mm_HandSolder, F.Cu at (93.8, 123.3)
- added C72: 100nF, Capacitor_SMD:C_1206_3216Metric_Pad1.33x1.80mm_HandSolder, F.Cu at (93.8, 126.6)
- added C73: 100nF, Capacitor_SMD:C_1206_3216Metric_Pad1.33x1.80mm_HandSolder, F.Cu at (99.8, 116.6)
- added C74: 100nF, Capacitor_SMD:C_1206_3216Metric_Pad1.33x1.80mm_HandSolder, F.Cu at (99.8, 119.9)
- added C75: 15pF, Capacitor_SMD:C_1206_3216Metric_Pad1.33x1.80mm_HandSolder, F.Cu at (99.8, 123.3)
- added C76: 15pF, Capacitor_SMD:C_1206_3216Metric_Pad1.33x1.80mm_HandSolder, F.Cu at (99.8, 126.6)
- added C77: 470pF, Capacitor_SMD:C_1206_3216Metric_Pad1.33x1.80mm_HandSolder, F.Cu at (105.8, 116.6)
- added C78: 10µF, Capacitor_SMD:C_1206_3216Metric_Pad1.33x1.80mm_HandSolder, F.Cu at (105.8, 119.9)
- added C79: 10µF, Capacitor_SMD:C_1206_3216Metric_Pad1.33x1.80mm_HandSolder, F.Cu at (105.8, 123.3)
- added C8: 100nF, Capacitor_SMD:C_1206_3216Metric_Pad1.33x1.80mm_HandSolder, F.Cu at (93.8, 104.5)
- added C80: 1µF, Capacitor_SMD:C_1206_3216Metric_Pad1.33x1.80mm_HandSolder, F.Cu at (105.8, 126.6)
- added C9: 100nF, Capacitor_SMD:C_1206_3216Metric_Pad1.33x1.80mm_HandSolder, F.Cu at (93.8, 107.9)
- added R1: 10k, Resistor_SMD:R_1206_3216Metric_Pad1.30x1.75mm_HandSolder, F.Cu at (103.0, 60.3)
- added R10: 10k, Resistor_SMD:R_1206_3216Metric_Pad1.30x1.75mm_HandSolder, F.Cu at (108.9, 66.9)
- added R11: 10k, Resistor_SMD:R_1206_3216Metric_Pad1.30x1.75mm_HandSolder, F.Cu at (108.9, 70.2)
- added R12: 10k, Resistor_SMD:R_1206_3216Metric_Pad1.30x1.75mm_HandSolder, F.Cu at (108.9, 73.5)
- added R13: 10k, Resistor_SMD:R_1206_3216Metric_Pad1.30x1.75mm_HandSolder, F.Cu at (108.9, 76.8)
- added R14: 10k, Resistor_SMD:R_1206_3216Metric_Pad1.30x1.75mm_HandSolder, F.Cu at (108.9, 80.1)
- added R15: 10k, Resistor_SMD:R_1206_3216Metric_Pad1.30x1.75mm_HandSolder, F.Cu at (46.0, 94.5)
- added R16: 10k, Resistor_SMD:R_1206_3216Metric_Pad1.30x1.75mm_HandSolder, F.Cu at (46.0, 97.8)
- added R17: 10k, Resistor_SMD:R_1206_3216Metric_Pad1.30x1.75mm_HandSolder, F.Cu at (46.0, 101.1)
- added R18: 10k, Resistor_SMD:R_1206_3216Metric_Pad1.30x1.75mm_HandSolder, F.Cu at (46.0, 104.4)
- added R19: 10k, Resistor_SMD:R_1206_3216Metric_Pad1.30x1.75mm_HandSolder, F.Cu at (46.0, 107.7)
- added R2: 10k, Resistor_SMD:R_1206_3216Metric_Pad1.30x1.75mm_HandSolder, F.Cu at (103.0, 63.6)
- added R20: 10k, Resistor_SMD:R_1206_3216Metric_Pad1.30x1.75mm_HandSolder, F.Cu at (46.0, 111.0)
- added R21: 10k, Resistor_SMD:R_1206_3216Metric_Pad1.30x1.75mm_HandSolder, F.Cu at (52.0, 94.5)
- added R22: 10k, Resistor_SMD:R_1206_3216Metric_Pad1.30x1.75mm_HandSolder, F.Cu at (52.0, 97.8)
- added R23: 10k, Resistor_SMD:R_1206_3216Metric_Pad1.30x1.75mm_HandSolder, F.Cu at (52.0, 101.1)
- added R24: 10k, Resistor_SMD:R_1206_3216Metric_Pad1.30x1.75mm_HandSolder, F.Cu at (52.0, 104.4)
- added R25: 10k, Resistor_SMD:R_1206_3216Metric_Pad1.30x1.75mm_HandSolder, F.Cu at (52.0, 107.7)
- added R26: 10k, Resistor_SMD:R_1206_3216Metric_Pad1.30x1.75mm_HandSolder, F.Cu at (52.0, 111.0)
- added R27: 10k, Resistor_SMD:R_1206_3216Metric_Pad1.30x1.75mm_HandSolder, F.Cu at (57.9, 94.5)
- added R28: 10k, Resistor_SMD:R_1206_3216Metric_Pad1.30x1.75mm_HandSolder, F.Cu at (57.9, 97.8)
- added R29: 10k, Resistor_SMD:R_1206_3216Metric_Pad1.30x1.75mm_HandSolder, F.Cu at (57.9, 101.1)
- added R3: 10k, Resistor_SMD:R_1206_3216Metric_Pad1.30x1.75mm_HandSolder, F.Cu at (103.0, 66.9)
- added R30: 10k, Resistor_SMD:R_1206_3216Metric_Pad1.30x1.75mm_HandSolder, F.Cu at (57.9, 104.4)
- added R31: 10k, Resistor_SMD:R_1206_3216Metric_Pad1.30x1.75mm_HandSolder, F.Cu at (57.9, 107.7)
- added R32: 10k, Resistor_SMD:R_1206_3216Metric_Pad1.30x1.75mm_HandSolder, F.Cu at (57.9, 111.0)
- added R33: 10k, Resistor_SMD:R_1206_3216Metric_Pad1.30x1.75mm_HandSolder, F.Cu at (63.9, 94.5)
- added R34: 10k, Resistor_SMD:R_1206_3216Metric_Pad1.30x1.75mm_HandSolder, F.Cu at (63.9, 97.8)
- added R35: 10k, Resistor_SMD:R_1206_3216Metric_Pad1.30x1.75mm_HandSolder, F.Cu at (74.6, 94.5)
- added R36: 10k, Resistor_SMD:R_1206_3216Metric_Pad1.30x1.75mm_HandSolder, F.Cu at (74.6, 97.8)
- added R37: 10k, Resistor_SMD:R_1206_3216Metric_Pad1.30x1.75mm_HandSolder, F.Cu at (74.6, 101.1)
- added R38: 10k, Resistor_SMD:R_1206_3216Metric_Pad1.30x1.75mm_HandSolder, F.Cu at (74.6, 104.4)
- added R39: 10k, Resistor_SMD:R_1206_3216Metric_Pad1.30x1.75mm_HandSolder, F.Cu at (74.6, 107.7)
- added R4: 10k, Resistor_SMD:R_1206_3216Metric_Pad1.30x1.75mm_HandSolder, F.Cu at (103.0, 70.2)
- added R40: 10k, Resistor_SMD:R_1206_3216Metric_Pad1.30x1.75mm_HandSolder, F.Cu at (74.6, 111.0)
- added R41: 10k, Resistor_SMD:R_1206_3216Metric_Pad1.30x1.75mm_HandSolder, F.Cu at (74.6, 114.3)
- added R42: 10k, Resistor_SMD:R_1206_3216Metric_Pad1.30x1.75mm_HandSolder, F.Cu at (74.6, 117.6)
- added R43: 10k, Resistor_SMD:R_1206_3216Metric_Pad1.30x1.75mm_HandSolder, F.Cu at (74.6, 120.9)
- added R44: 10M, Resistor_SMD:R_1206_3216Metric_Pad1.30x1.75mm_HandSolder, F.Cu at (63.9, 101.1)
- added R45: 10M, Resistor_SMD:R_1206_3216Metric_Pad1.30x1.75mm_HandSolder, F.Cu at (63.9, 104.4)
- added R46: 10M, Resistor_SMD:R_1206_3216Metric_Pad1.30x1.75mm_HandSolder, F.Cu at (63.9, 107.7)
- added R47: 10M, Resistor_SMD:R_1206_3216Metric_Pad1.30x1.75mm_HandSolder, F.Cu at (63.9, 111.0)
- added R48: 5.1k, Resistor_SMD:R_1206_3216Metric_Pad1.30x1.75mm_HandSolder, F.Cu at (111.8, 116.6)
- added R49: 5.1k, Resistor_SMD:R_1206_3216Metric_Pad1.30x1.75mm_HandSolder, F.Cu at (111.8, 119.9)
- added R5: 10k, Resistor_SMD:R_1206_3216Metric_Pad1.30x1.75mm_HandSolder, F.Cu at (103.0, 73.5)
- added R50: 10k, Resistor_SMD:R_1206_3216Metric_Pad1.30x1.75mm_HandSolder, F.Cu at (111.8, 123.2)
- added R51: 1k, Resistor_SMD:R_1206_3216Metric_Pad1.30x1.75mm_HandSolder, F.Cu at (111.8, 126.5)
- added R6: 10k, Resistor_SMD:R_1206_3216Metric_Pad1.30x1.75mm_HandSolder, F.Cu at (103.0, 76.8)
- added R7: 10k, Resistor_SMD:R_1206_3216Metric_Pad1.30x1.75mm_HandSolder, F.Cu at (103.0, 80.1)
- added R8: 10k, Resistor_SMD:R_1206_3216Metric_Pad1.30x1.75mm_HandSolder, F.Cu at (108.9, 60.3)
- added R9: 10k, Resistor_SMD:R_1206_3216Metric_Pad1.30x1.75mm_HandSolder, F.Cu at (108.9, 63.6)
- added U1: ~, Package_TO_SOT_SMD:SOT-23-5, F.Cu at (97.4, 61.0)
- added U10: ~, Package_TO_SOT_SMD:SOT-23-5, F.Cu at (45.6, 124.3)
- added U100: AD5160, Package_TO_SOT_SMD:SOT-23-8, F.Cu at (45.6, 61.0)
- added U101: AD5160, Package_TO_SOT_SMD:SOT-23-8, F.Cu at (45.6, 65.6)
- added U102: AD5160, Package_TO_SOT_SMD:SOT-23-8, F.Cu at (45.6, 70.2)
- added U103: AD5160, Package_TO_SOT_SMD:SOT-23-8, F.Cu at (45.6, 74.8)
- added U104: AD5160, Package_TO_SOT_SMD:SOT-23-8, F.Cu at (45.6, 79.4)
- added U105: AD5160, Package_TO_SOT_SMD:SOT-23-8, F.Cu at (45.6, 84.0)
- added U106: AD5160, Package_TO_SOT_SMD:SOT-23-8, F.Cu at (45.6, 88.6)
- added U107: AD5160, Package_TO_SOT_SMD:SOT-23-8, F.Cu at (50.8, 61.0)
- added U108: AD5160, Package_TO_SOT_SMD:SOT-23-8, F.Cu at (50.8, 65.6)
- added U109: AD5160, Package_TO_SOT_SMD:SOT-23-8, F.Cu at (50.8, 70.2)
- added U11: ~, Package_TO_SOT_SMD:SOT-23-5, F.Cu at (45.6, 128.9)
- added U110: AD5160, Package_TO_SOT_SMD:SOT-23-8, F.Cu at (50.8, 74.8)
- added U111: AD5160, Package_TO_SOT_SMD:SOT-23-8, F.Cu at (50.8, 79.4)
- added U112: AD5160, Package_TO_SOT_SMD:SOT-23-8, F.Cu at (50.8, 84.0)
- added U113: AD5160, Package_TO_SOT_SMD:SOT-23-8, F.Cu at (50.8, 88.6)
- added U114: AD5160, Package_TO_SOT_SMD:SOT-23-8, F.Cu at (55.9, 61.0)
- added U115: AD5160, Package_TO_SOT_SMD:SOT-23-8, F.Cu at (55.9, 65.6)
- added U116: AD5160, Package_TO_SOT_SMD:SOT-23-8, F.Cu at (55.9, 70.2)
- added U117: AD5160, Package_TO_SOT_SMD:SOT-23-8, F.Cu at (55.9, 74.8)
- added U118: AD5160, Package_TO_SOT_SMD:SOT-23-8, F.Cu at (55.9, 79.4)
- added U119: AD5160, Package_TO_SOT_SMD:SOT-23-8, F.Cu at (55.9, 84.0)
- added U12: ~, Package_TO_SOT_SMD:SOT-23-5, F.Cu at (50.8, 115.1)
- added U120: AD5160, Package_TO_SOT_SMD:SOT-23-8, F.Cu at (55.9, 88.6)
- added U121: AD5160, Package_TO_SOT_SMD:SOT-23-8, F.Cu at (61.1, 61.0)
- added U122: AD5160, Package_TO_SOT_SMD:SOT-23-8, F.Cu at (61.1, 65.6)
- added U123: AD5160, Package_TO_SOT_SMD:SOT-23-8, F.Cu at (61.1, 70.2)
- added U124: AD5160, Package_TO_SOT_SMD:SOT-23-8, F.Cu at (61.1, 74.8)
- added U125: AD5160, Package_TO_SOT_SMD:SOT-23-8, F.Cu at (61.1, 79.4)
- added U126: AD5160, Package_TO_SOT_SMD:SOT-23-8, F.Cu at (61.1, 84.0)
- added U127: AD5160, Package_TO_SOT_SMD:SOT-23-8, F.Cu at (61.1, 88.6)
- added U128: AD5160, Package_TO_SOT_SMD:SOT-23-8, F.Cu at (66.2, 61.0)
- added U129: AD5160, Package_TO_SOT_SMD:SOT-23-8, F.Cu at (66.2, 65.6)
- added U13: ~, Package_TO_SOT_SMD:SOT-23-5, F.Cu at (50.8, 119.7)
- added U130: AD5160, Package_TO_SOT_SMD:SOT-23-8, F.Cu at (66.2, 70.2)
- added U131: AD5160, Package_TO_SOT_SMD:SOT-23-8, F.Cu at (66.2, 74.8)
- added U14: ~, Package_TO_SOT_SMD:SOT-23-5, F.Cu at (50.8, 124.3)
- added U15: ~, Package_TO_SOT_SMD:SOT-23-5, F.Cu at (50.8, 128.9)
- added U16: ~, Package_TO_SOT_SMD:SOT-23-5, F.Cu at (55.9, 115.1)
- added U17: ~, Package_TO_SOT_SMD:SOT-23-5, F.Cu at (55.9, 119.7)
- added U18: ~, Package_TO_SOT_SMD:SOT-23-5, F.Cu at (55.9, 124.3)
- added U19: ~, Package_TO_SOT_SMD:SOT-23-5, F.Cu at (55.9, 128.9)
- added U2: TLV9061xDBV, Package_TO_SOT_SMD:SOT-23-5, F.Cu at (111.4, 130.6)
- added U20: ~, Package_TO_SOT_SMD:SOT-23-5, F.Cu at (61.1, 115.1)
- added U21: ~, Package_TO_SOT_SMD:SOT-23-5, F.Cu at (61.1, 119.7)
- added U22: ~, Package_TO_SOT_SMD:SOT-23-5, F.Cu at (61.1, 124.3)
- added U23: ~, Package_TO_SOT_SMD:SOT-23-5, F.Cu at (61.1, 128.9)
- added U24: ~, Package_TO_SOT_SMD:SOT-23-5, F.Cu at (86.2, 95.2)
- added U25: ~, Package_TO_SOT_SMD:SOT-23-5, F.Cu at (86.2, 99.8)
- added U26: ~, Package_TO_SOT_SMD:SOT-23-5, F.Cu at (86.2, 104.5)
- added U27: ~, Package_TO_SOT_SMD:SOT-23-5, F.Cu at (86.2, 109.1)
- added U3: ~, Package_TO_SOT_SMD:SOT-23-5, F.Cu at (97.4, 65.6)
- added U4: ~, Package_TO_SOT_SMD:SOT-23-5, F.Cu at (97.4, 70.3)
- added U5: ~, Package_TO_SOT_SMD:SOT-23-5, F.Cu at (97.4, 74.9)
- added U6: ~, Package_TO_SOT_SMD:SOT-23-5, F.Cu at (97.4, 79.5)
- added U7: ~, Package_TO_SOT_SMD:SOT-23-5, F.Cu at (97.4, 84.1)
- added U8: ~, Package_TO_SOT_SMD:SOT-23-5, F.Cu at (45.6, 115.1)
- added U9: ~, Package_TO_SOT_SMD:SOT-23-5, F.Cu at (45.6, 119.7)
- added U92: ~, Package_TO_SOT_SMD:SOT-23-5, F.Cu at (86.2, 113.7)
- U36, U37, U38, U39: value AD5160 -> 74HC595
- U40: value AD5160 -> RP2040; footprint Package_TO_SOT_SMD:SOT-23-8 -> Package_DFN_QFN:QFN-56-1EP_7x7mm_P0.4mm_EP3.2x3.2mm
- U41: value AD5160 -> W25Q128JVS; footprint Package_TO_SOT_SMD:SOT-23-8 -> Package_SO:SOIC-8_5.3x5.3mm_P1.27mm
- U42: value AD5160 -> MIC5219-3.3YM5; footprint Package_TO_SOT_SMD:SOT-23-8 -> Package_TO_SOT_SMD:SOT-23-5
- U43: value AD5160 -> TLV9061xDBV; footprint Package_TO_SOT_SMD:SOT-23-8 -> Package_TO_SOT_SMD:SOT-23-5
Connections:
- U28 pad 2: unconnected-(U28-V_{DD}-Pad2) -> VCC
- U28 pad 4: unconnected-(U28-CLK-Pad4) -> CLK
- U28 pad 5: unconnected-(U28-SDI-Pad5) -> SDI
- U28 pad 6: unconnected-(U28-~{CS}-Pad6) -> Wo1
- U28 pad 7: unconnected-(U28-B-Pad7) -> VREF
- U29 pad 2: unconnected-(U29-V_{DD}-Pad2) -> VCC
- U29 pad 4: unconnected-(U29-CLK-Pad4) -> CLK
- U29 pad 5: unconnected-(U29-SDI-Pad5) -> SDI
- U29 pad 6: unconnected-(U29-~{CS}-Pad6) -> Wo1_neg
- U29 pad 7: Net-(U28-A) -> VREF
- U29 pad 8: unconnected-(U29-A-Pad8) -> Net-(U28-A)
- U30 pad 2: unconnected-(U30-V_{DD}-Pad2) -> VCC
- U30 pad 4: unconnected-(U30-CLK-Pad4) -> CLK
- U30 pad 5: unconnected-(U30-SDI-Pad5) -> SDI
- U30 pad 6: unconnected-(U30-~{CS}-Pad6) -> Wo2
- U30 pad 7: unconnected-(U30-B-Pad7) -> VREF
- U31 pad 2: unconnected-(U31-V_{DD}-Pad2) -> VCC
- U31 pad 4: unconnected-(U31-CLK-Pad4) -> CLK
- U31 pad 5: unconnected-(U31-SDI-Pad5) -> SDI
- U31 pad 6: unconnected-(U31-~{CS}-Pad6) -> Wo2_neg
- U31 pad 7: Net-(U28-A) -> VREF
- U31 pad 8: unconnected-(U31-A-Pad8) -> Net-(U28-A)
- U32 pad 2: unconnected-(U32-V_{DD}-Pad2) -> VCC
- U32 pad 4: unconnected-(U32-CLK-Pad4) -> CLK
- U32 pad 5: unconnected-(U32-SDI-Pad5) -> SDI
- U32 pad 6: unconnected-(U32-~{CS}-Pad6) -> Wo3
- U32 pad 7: unconnected-(U32-B-Pad7) -> VREF
- U33 pad 2: unconnected-(U33-V_{DD}-Pad2) -> VCC
- U33 pad 4: unconnected-(U33-CLK-Pad4) -> CLK
- U33 pad 5: unconnected-(U33-SDI-Pad5) -> SDI
- U33 pad 6: unconnected-(U33-~{CS}-Pad6) -> Wo3_neg
- U33 pad 7: Net-(U28-A) -> VREF
- U33 pad 8: unconnected-(U33-A-Pad8) -> Net-(U28-A)
- U34 pad 2: unconnected-(U34-V_{DD}-Pad2) -> VCC
- U34 pad 4: unconnected-(U34-CLK-Pad4) -> CLK
- U34 pad 5: unconnected-(U34-SDI-Pad5) -> SDI
- U34 pad 6: unconnected-(U34-~{CS}-Pad6) -> Wo4
- U34 pad 7: unconnected-(U34-B-Pad7) -> VREF
- U35 pad 2: unconnected-(U35-V_{DD}-Pad2) -> VCC
- U35 pad 4: unconnected-(U35-CLK-Pad4) -> CLK
- U35 pad 5: unconnected-(U35-SDI-Pad5) -> SDI
- U35 pad 6: unconnected-(U35-~{CS}-Pad6) -> Wo4_neg
- U35 pad 7: Net-(U28-A) -> VREF
- U35 pad 8: unconnected-(U35-A-Pad8) -> Net-(U28-A)
- U36 pad 1: +Vh1 -> CS21_neg
- U36 pad 2: unconnected-(U36-V_{DD}-Pad2) -> CS31_neg
- U36 pad 3: GND -> CS41_neg
- U36 pad 4: unconnected-(U36-CLK-Pad4) -> CS12_neg
- U36 pad 5: unconnected-(U36-SDI-Pad5) -> CS22_neg
- U36 pad 6: unconnected-(U36-~{CS}-Pad6) -> CS32_neg
- U36 pad 7: unconnected-(U36-B-Pad7) -> CS42_neg
- U36 pad 8: cbar1 -> GND
- U37 pad 1: +Vh1 -> CS23_neg
- U37 pad 2: unconnected-(U37-V_{DD}-Pad2) -> CS33_neg
- U37 pad 3: GND -> CS43_neg
- U37 pad 4: unconnected-(U37-CLK-Pad4) -> CS11_neg_h
- U37 pad 5: unconnected-(U37-SDI-Pad5) -> CS21_neg_h
- U37 pad 6: unconnected-(U37-~{CS}-Pad6) -> CS31_neg_h
- U37 pad 7: unconnected-(U37-B-Pad7) -> CS41_neg_h
- U37 pad 8: cbar2 -> GND
- U38 pad 1: +Vh1 -> CS22_neg_h
- U38 pad 2: unconnected-(U38-V_{DD}-Pad2) -> CS32_neg_h
- U38 pad 3: GND -> CS42_neg_h
- U38 pad 4: unconnected-(U38-CLK-Pad4) -> CS13_neg_h
- U38 pad 5: unconnected-(U38-SDI-Pad5) -> CS23_neg_h
- U38 pad 6: unconnected-(U38-~{CS}-Pad6) -> CS33_neg_h
- U38 pad 7: unconnected-(U38-B-Pad7) -> CS43_neg_h
- U38 pad 8: cbar3 -> GND
- U39 pad 1: +Vh1 -> CS24_neg_h
- U39 pad 2: unconnected-(U39-V_{DD}-Pad2) -> CS34_neg_h
- U39 pad 3: GND -> CS44_neg_h
- U39 pad 4: unconnected-(U39-CLK-Pad4) -> Wo1_neg
- U39 pad 5: unconnected-(U39-SDI-Pad5) -> Wo2_neg
- U39 pad 6: unconnected-(U39-~{CS}-Pad6) -> Wo3_neg
- U39 pad 7: unconnected-(U39-B-Pad7) -> Wo4_neg
- U39 pad 8: cbar4 -> GND
- U40 pad 1: -Vh1 -> VCC
- U40 pad 3: GND -> unconnected-(U40-GPIO1-Pad3)
- U40 pad 4: unconnected-(U40-CLK-Pad4) -> SRCLK
- U40 pad 5: unconnected-(U40-SDI-Pad5) -> ser
- U40 pad 6: unconnected-(U40-~{CS}-Pad6) -> RCLK
- U40 pad 7: cbar1 -> unconnected-(U40-GPIO5-Pad7)
- U41 pad 1: -Vh1 -> Net-(U40-QSPI_SS)
- U41 pad 2: unconnected-(U41-V_{DD}-Pad2) -> Net-(U40-QSPI_SD1)
- U41 pad 3: GND -> Net-(U40-QSPI_SD2)
- U41 pad 4: unconnected-(U41-CLK-Pad4) -> GND
- U41 pad 5: unconnected-(U41-SDI-Pad5) -> Net-(U40-QSPI_SD0)
- U41 pad 6: unconnected-(U41-~{CS}-Pad6) -> Net-(U40-QSPI_SCLK)
- U41 pad 7: cbar2 -> Net-(U40-QSPI_SD3)
- U41 pad 8: unconnected-(U41-A-Pad8) -> VCC
- U42 pad 1: -Vh1 -> Net-(U42-EN)
- U42 pad 2: unconnected-(U42-V_{DD}-Pad2) -> GND
- U42 pad 3: GND -> Net-(U42-EN)
- U42 pad 4: unconnected-(U42-CLK-Pad4) -> Net-(U42-BP)
- U42 pad 5: unconnected-(U42-SDI-Pad5) -> VCC
- U43 pad 1: -Vh1 -> -Vu1
- U43 pad 2: unconnected-(U43-V_{DD}-Pad2) -> GND
- U43 pad 3: GND -> VREF
- U43 pad 4: unconnected-(U43-CLK-Pad4) -> Net-(U43--)
- U43 pad 5: unconnected-(U43-SDI-Pad5) -> VCC
- U60 pad 2: unconnected-(U60-V_{DD}-Pad2) -> VCC
- U60 pad 4: unconnected-(U60-CLK-Pad4) -> CLK
- U60 pad 5: unconnected-(U60-SDI-Pad5) -> SDI
- U60 pad 6: unconnected-(U60-~{CS}-Pad6) -> CS11
- U60 pad 7: unconnected-(U60-B-Pad7) -> VREF
- U61 pad 2: unconnected-(U61-V_{DD}-Pad2) -> VCC
- U61 pad 4: unconnected-(U61-CLK-Pad4) -> CLK
- U61 pad 5: unconnected-(U61-SDI-Pad5) -> SDI
- U61 pad 6: unconnected-(U61-~{CS}-Pad6) -> CS21
- U61 pad 7: unconnected-(U61-B-Pad7) -> VREF
- U62 pad 2: unconnected-(U62-V_{DD}-Pad2) -> VCC
- U62 pad 4: unconnected-(U62-CLK-Pad4) -> CLK
- U62 pad 5: unconnected-(U62-SDI-Pad5) -> SDI
- U62 pad 6: unconnected-(U62-~{CS}-Pad6) -> CS31
- U62 pad 7: unconnected-(U62-B-Pad7) -> VREF
- U63 pad 2: unconnected-(U63-V_{DD}-Pad2) -> VCC
- U63 pad 4: unconnected-(U63-CLK-Pad4) -> CLK
- U63 pad 5: unconnected-(U63-SDI-Pad5) -> SDI
- U63 pad 6: unconnected-(U63-~{CS}-Pad6) -> CS41
- U63 pad 7: unconnected-(U63-B-Pad7) -> VREF
- U64 pad 2: unconnected-(U64-V_{DD}-Pad2) -> VCC
- U64 pad 4: unconnected-(U64-CLK-Pad4) -> CLK
- U64 pad 5: unconnected-(U64-SDI-Pad5) -> SDI
- U64 pad 6: unconnected-(U64-~{CS}-Pad6) -> CS11_neg
- U64 pad 7: cbar1 -> VREF
- U64 pad 8: unconnected-(U64-A-Pad8) -> cbar1
- U65 pad 2: unconnected-(U65-V_{DD}-Pad2) -> VCC
- U65 pad 4: unconnected-(U65-CLK-Pad4) -> CLK
- U65 pad 5: unconnected-(U65-SDI-Pad5) -> SDI
- U65 pad 6: unconnected-(U65-~{CS}-Pad6) -> CS21_neg
- U65 pad 7: cbar2 -> VREF
- U65 pad 8: unconnected-(U65-A-Pad8) -> cbar2
- U66 pad 2: unconnected-(U66-V_{DD}-Pad2) -> VCC
- U66 pad 4: unconnected-(U66-CLK-Pad4) -> CLK
- U66 pad 5: unconnected-(U66-SDI-Pad5) -> SDI
- U66 pad 6: unconnected-(U66-~{CS}-Pad6) -> CS31_neg
- U66 pad 7: cbar3 -> VREF
- U66 pad 8: unconnected-(U66-A-Pad8) -> cbar3
- U67 pad 2: unconnected-(U67-V_{DD}-Pad2) -> VCC
- U67 pad 4: unconnected-(U67-CLK-Pad4) -> CLK
- U67 pad 5: unconnected-(U67-SDI-Pad5) -> SDI
- U67 pad 6: unconnected-(U67-~{CS}-Pad6) -> CS41_neg
- U67 pad 7: cbar4 -> VREF
- U67 pad 8: unconnected-(U67-A-Pad8) -> cbar4
- U68 pad 2: unconnected-(U68-V_{DD}-Pad2) -> VCC
- U68 pad 4: unconnected-(U68-CLK-Pad4) -> CLK
- U68 pad 5: unconnected-(U68-SDI-Pad5) -> SDI
- U68 pad 6: unconnected-(U68-~{CS}-Pad6) -> CS12
- U68 pad 7: unconnected-(U68-B-Pad7) -> VREF
- U69 pad 2: unconnected-(U69-V_{DD}-Pad2) -> VCC
- U69 pad 4: unconnected-(U69-CLK-Pad4) -> CLK
- U69 pad 5: unconnected-(U69-SDI-Pad5) -> SDI
- U69 pad 6: unconnected-(U69-~{CS}-Pad6) -> CS22
- U69 pad 7: unconnected-(U69-B-Pad7) -> VREF
- U70 pad 2: unconnected-(U70-V_{DD}-Pad2) -> VCC
- U70 pad 4: unconnected-(U70-CLK-Pad4) -> CLK
- U70 pad 5: unconnected-(U70-SDI-Pad5) -> SDI
- U70 pad 6: unconnected-(U70-~{CS}-Pad6) -> CS32
- U70 pad 7: unconnected-(U70-B-Pad7) -> VREF
- U71 pad 2: unconnected-(U71-V_{DD}-Pad2) -> VCC
- U71 pad 4: unconnected-(U71-CLK-Pad4) -> CLK
- U71 pad 5: unconnected-(U71-SDI-Pad5) -> SDI
- U71 pad 6: unconnected-(U71-~{CS}-Pad6) -> CS42
- U71 pad 7: unconnected-(U71-B-Pad7) -> VREF
- U72 pad 2: unconnected-(U72-V_{DD}-Pad2) -> VCC
- U72 pad 4: unconnected-(U72-CLK-Pad4) -> CLK
- U72 pad 5: unconnected-(U72-SDI-Pad5) -> SDI
- U72 pad 6: unconnected-(U72-~{CS}-Pad6) -> CS12_neg
- U72 pad 7: cbar1 -> VREF
- U72 pad 8: unconnected-(U72-A-Pad8) -> cbar1
- U73 pad 2: unconnected-(U73-V_{DD}-Pad2) -> VCC
- U73 pad 4: unconnected-(U73-CLK-Pad4) -> CLK
- U73 pad 5: unconnected-(U73-SDI-Pad5) -> SDI
- U73 pad 6: unconnected-(U73-~{CS}-Pad6) -> CS22_neg
- U73 pad 7: cbar2 -> VREF
- U73 pad 8: unconnected-(U73-A-Pad8) -> cbar2
- U74 pad 2: unconnected-(U74-V_{DD}-Pad2) -> VCC
- U74 pad 4: unconnected-(U74-CLK-Pad4) -> CLK
- U74 pad 5: unconnected-(U74-SDI-Pad5) -> SDI
- U74 pad 6: unconnected-(U74-~{CS}-Pad6) -> CS32_neg
- U74 pad 7: cbar3 -> VREF
- U74 pad 8: unconnected-(U74-A-Pad8) -> cbar3
- U75 pad 2: unconnected-(U75-V_{DD}-Pad2) -> VCC
- U75 pad 4: unconnected-(U75-CLK-Pad4) -> CLK
- U75 pad 5: unconnected-(U75-SDI-Pad5) -> SDI
- U75 pad 6: unconnected-(U75-~{CS}-Pad6) -> CS42_neg
- U75 pad 7: cbar4 -> VREF
- U75 pad 8: unconnected-(U75-A-Pad8) -> cbar4
- U76 pad 2: unconnected-(U76-V_{DD}-Pad2) -> VCC
- U76 pad 4: unconnected-(U76-CLK-Pad4) -> CLK
- U76 pad 5: unconnected-(U76-SDI-Pad5) -> SDI
- U76 pad 6: unconnected-(U76-~{CS}-Pad6) -> CS13
- U76 pad 7: unconnected-(U76-B-Pad7) -> VREF
- U77 pad 2: unconnected-(U77-V_{DD}-Pad2) -> VCC
- U77 pad 4: unconnected-(U77-CLK-Pad4) -> CLK
- U77 pad 5: unconnected-(U77-SDI-Pad5) -> SDI
- U77 pad 6: unconnected-(U77-~{CS}-Pad6) -> CS23
- U77 pad 7: unconnected-(U77-B-Pad7) -> VREF
- U78 pad 2: unconnected-(U78-V_{DD}-Pad2) -> VCC
- U78 pad 4: unconnected-(U78-CLK-Pad4) -> CLK
- U78 pad 5: unconnected-(U78-SDI-Pad5) -> SDI
- U78 pad 6: unconnected-(U78-~{CS}-Pad6) -> CS33
- U78 pad 7: unconnected-(U78-B-Pad7) -> VREF
- U79 pad 2: unconnected-(U79-V_{DD}-Pad2) -> VCC
- U79 pad 4: unconnected-(U79-CLK-Pad4) -> CLK
- U79 pad 5: unconnected-(U79-SDI-Pad5) -> SDI
- U79 pad 6: unconnected-(U79-~{CS}-Pad6) -> CS43
- U79 pad 7: unconnected-(U79-B-Pad7) -> VREF
- U80 pad 2: unconnected-(U80-V_{DD}-Pad2) -> VCC
- U80 pad 4: unconnected-(U80-CLK-Pad4) -> CLK
- U80 pad 5: unconnected-(U80-SDI-Pad5) -> SDI
- U80 pad 6: unconnected-(U80-~{CS}-Pad6) -> CS13_neg
- U80 pad 7: cbar1 -> VREF
- U80 pad 8: unconnected-(U80-A-Pad8) -> cbar1
- U81 pad 2: unconnected-(U81-V_{DD}-Pad2) -> VCC
- U81 pad 4: unconnected-(U81-CLK-Pad4) -> CLK
- U81 pad 5: unconnected-(U81-SDI-Pad5) -> SDI
- U81 pad 6: unconnected-(U81-~{CS}-Pad6) -> CS23_neg
- U81 pad 7: cbar2 -> VREF
- U81 pad 8: unconnected-(U81-A-Pad8) -> cbar2
- U82 pad 2: unconnected-(U82-V_{DD}-Pad2) -> VCC
- U82 pad 4: unconnected-(U82-CLK-Pad4) -> CLK
- U82 pad 5: unconnected-(U82-SDI-Pad5) -> SDI
- U82 pad 6: unconnected-(U82-~{CS}-Pad6) -> CS33_neg
- U82 pad 7: cbar3 -> VREF
- U82 pad 8: unconnected-(U82-A-Pad8) -> cbar3
- U83 pad 2: unconnected-(U83-V_{DD}-Pad2) -> VCC
- U83 pad 4: unconnected-(U83-CLK-Pad4) -> CLK
- U83 pad 5: unconnected-(U83-SDI-Pad5) -> SDI
- U83 pad 6: unconnected-(U83-~{CS}-Pad6) -> CS43_neg
- U83 pad 7: cbar4 -> VREF
- U83 pad 8: unconnected-(U83-A-Pad8) -> cbar4
