File: analog_NN.kicad_pcb (KiCad board)
At the start: 4 copper layers, 230 parts, among them J1 Conn_01x01, J2 Conn_01x01, J3 Conn_01x01, J4 Conn_01x01, J5 Conn_01x01, J6 Conn_01x01, J7 Conn_01x01, U100 AD5160, U101 AD5160, U102 AD5160, U103 AD5160, U104 AD5160, U105 AD5160, U106 AD5160, U107 AD5160, U108 AD5160, U109 AD5160, U110 AD5160, U111 AD5160, U112 AD5160, U113 AD5160, U114 AD5160, U115 AD5160, U116 AD5160, U117 AD5160, U118 AD5160, U119 AD5160, U120 AD5160, U121 AD5160, U122 AD5160, U123 AD5160, U124 AD5160, U125 AD5160, U126 AD5160, U127 AD5160, U128 AD5160, U129 AD5160, U130 AD5160, U131 AD5160, U132 TLV9061xDBV, U28 AD5160, U29 AD5160, U30 AD5160, U31 AD5160, U32 AD5160, U33 AD5160, U34 AD5160, U35 AD5160, U36 74HC595, U37 74HC595, U38 74HC595, U39 74HC595, U43 TLV9061xDBV, U60 AD5160, U61 AD5160, U62 AD5160, U63 AD5160, U64 AD5160, U65 AD5160, U66 AD5160, U67 AD5160, U68 AD5160, U69 AD5160, U70 AD5160, U71 AD5160, U72 AD5160, U73 AD5160, U74 AD5160, U75 AD5160, U76 AD5160, U77 AD5160, U78 AD5160, U79 AD5160, U80 AD5160, U81 AD5160, U82 AD5160, U83 AD5160, U93 74HC595, U94 74HC595, U95 74HC595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

Commit message: Updated: schematic
Parts:
- moved R14 257.4 mm to (32.1, 122.0), turned to 180 degrees
- moved R12 256.5 mm to (32.0, 105.4), turned to 180 degrees
- moved R8 250.7 mm to (31.4, 77.8), turned to 180 degrees
- moved R13 250.6 mm to (38.8, 117.2), turned to 180 degrees
- moved R10 249.9 mm to (32.0, 91.4), turned to 180 degrees
- moved R11 249.3 mm to (39.1, 101.3), turned to 180 degrees
- moved R7 243.2 mm to (38.9, 74.2), turned to 180 degrees
- moved R9 242.9 mm to (39.1, 87.6), turned to 180 degrees
- moved U7 234.5 mm to (39.3, 121.9), turned to 180 degrees
- moved U6 233.2 mm to (39.1, 106.1), turned to 180 degrees
- moved U4 227.3 mm to (38.8, 78.8), turned to 180 degrees
- moved U5 226.8 mm to (39.0, 92.2), turned to 180 degrees
- moved C28 215.6 mm to (76.8, 77.4), turned to 90 degrees
- moved C21 209.8 mm to (76.5, 67.4), turned to 90 degrees
- moved C20 209.5 mm to (76.7, 56.4), turned to 90 degrees
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Routing:
- net VDD: track 3.10 -> 253.1 mm, vias 2 -> 7
- net GND: track 3.07 -> 227.1 mm, vias 2 -> 63
- net cbar1: track 0.00 -> 12.2 mm
- net Net-(U3--): track 0.00 -> 9.92 mm
- net -Vu3: track 0.00 -> 9.67 mm
- net Net-(U7--): track 0.00 -> 9.13 mm
- net Net-(U4--): track 0.00 -> 8.62 mm
- net Net-(U6--): track 0.00 -> 8.59 mm
- net -Vh4: track 0.00 -> 8.42 mm
- net -Vh3: track 0.00 -> 8.34 mm
- net -Vh2: track 0.00 -> 8.33 mm
- net Net-(U5--): track 0.00 -> 8.14 mm
- net VREF: track 3.10 -> 10.7 mm, vias 2 -> 7
- net Vu3: track 0.00 -> 6.14 mm

Commit message: Updated: pcb
Parts:
- moved SDI 238.5 mm to (57.5, 17.8)
- moved CLK 234.5 mm to (57.6, 23.2)
- moved U94 102.3 mm to (149.9, 67.3)
- moved U37 66.1 mm to (149.7, 52.9)
- moved U36 58.3 mm to (147.1, 36.7)
- moved U93 31.9 mm to (147.1, 25.8)
- moved U38 19.0 mm to (223.8, 55.6)
- moved U95 17.3 mm to (250.8, 53.2)
- moved U131 17.2 mm to (128.3, 158.7)
- moved C60 17.2 mm to (133.0, 159.0)
- moved U129 17.0 mm to (98.7, 158.9)
- moved C58 17.0 mm to (103.7, 159.1)
- moved C59 17.0 mm to (119.2, 159.0)
- moved U130 17.0 mm to (114.0, 158.7)
- moved U121 16.9 mm to (98.7, 138.7)
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- renumbered J5 to CLK, J6 to SDI
Connections:
- U37 pad 10: VCC -> VDD
- U38 pad 10: VCC -> VDD
- U39 pad 10: VCC -> VDD
- U93 pad 10: VCC -> VDD
- U94 pad 10: VCC -> VDD
- U95 pad 10: VCC -> VDD
- U96 pad 10: VCC -> VDD
Routing:
- net SDI: track 0.00 -> 1299.8 mm, vias 0 -> 114
- net CLK: track 0.00 -> 1229.4 mm, vias 0 -> 26
- net VREF: track 10.7 -> 272.1 mm, vias 7 -> 24
- net cbar2: track 0.00 -> 185.1 mm, vias 0 -> 24
- net cbar3: track 0.00 -> 179.1 mm, vias 0 -> 24
- net cbar4: track 0.00 -> 172.4 mm, vias 0 -> 24
- net cbar1: track 12.2 -> 182.7 mm, vias 0 -> 24
- net CS11_neg: track 0.00 -> 110.2 mm, vias 0 -> 2
- net CS31_neg: track 0.00 -> 102.2 mm, vias 0 -> 2
- net CS22_neg: track 0.00 -> 91.3 mm, vias 0 -> 2
- net CS12: track 0.00 -> 88.6 mm, vias 0 -> 2
- net CS12_neg: track 0.00 -> 88.5 mm, vias 0 -> 2
- net CS11: track 0.00 -> 83.1 mm, vias 0 -> 2
- net CS32: track 0.00 -> 81.8 mm, vias 0 -> 2
- net CS22: track 0.00 -> 75.4 mm, vias 0 -> 2
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Other:
- board text added: "AD5160"
- board text added: "C5"
- board text added: "C6"
- board text added: "C7"

Commit message: Updated: pcb
Parts:
- moved U96 159.8 mm to (146.4, 144.3)
- moved U39 145.4 mm to (146.4, 155.1)
- moved U95 114.5 mm to (146.6, 100.7)
- moved U38 95.3 mm to (146.6, 111.4)
- moved U37 20.0 mm to (147.2, 72.7)
- moved U94 5.84 mm to (147.2, 62.1)
Routing:
- net VREF: track 272.1 -> 758.8 mm, vias 24 -> 71
- net CS13_neg: track 0.00 -> 123.5 mm, vias 0 -> 2
- net CS33_neg: track 0.00 -> 111.0 mm, vias 0 -> 6
- net CS11_h: track 0.00 -> 101.2 mm, vias 0 -> 2
- net CS13: track 0.00 -> 100.6 mm, vias 0 -> 2
- net CS13_h: track 0.00 -> 97.2 mm, vias 0 -> 2
- net CS23: track 0.00 -> 91.5 mm, vias 0 -> 2
- net CS23_neg: track 0.00 -> 87.2 mm, vias 0 -> 4
- net CS11_neg_h: track 0.00 -> 83.4 mm, vias 0 -> 2
- net CS21_h: track 0.00 -> 70.9 mm, vias 0 -> 2
- net CS21_neg_h: track 0.00 -> 66.9 mm, vias 0 -> 2
- net CS22_h: track 0.00 -> 55.9 mm, vias 0 -> 2
- net CS31_h: track 0.00 -> 54.6 mm, vias 0 -> 2
- net CS31_neg_h: track 0.00 -> 50.1 mm, vias 0 -> 2
- net CS33: track 0.00 -> 49.5 mm, vias 0 -> 2
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
Commit message: Updated: cross bar
Parts:
- moved SDI 14.9 mm to (72.4, 17.8)
- moved CLK 14.9 mm to (72.5, 23.2)
Routing:
- net CS12_h: track 0.00 -> 177.9 mm, vias 0 -> 2
- net CS12_neg_h: track 0.00 -> 169.3 mm, vias 0 -> 4
- net CS13_neg_h: track 0.00 -> 121.6 mm, vias 0 -> 2
- net CS14_h: track 0.00 -> 118.1 mm, vias 0 -> 2
- net CS23_neg_h: track 0.00 -> 116.0 mm, vias 0 -> 4
- net CS33_neg_h: track 0.00 -> 105.9 mm, vias 0 -> 4
- net CS14_neg_h: track 0.00 -> 104.4 mm, vias 0 -> 4
- net CS33_h: track 0.00 -> 84.2 mm, vias 0 -> 2
- net CS23_h: track 0.00 -> 74.6 mm, vias 0 -> 4
- net CS34_neg_h: track 0.00 -> 71.5 mm, vias 0 -> 6
- net CS24_neg_h: track 0.00 -> 69.3 mm, vias 0 -> 6
- net CS32_neg_h: track 0.00 -> 62.1 mm, vias 0 -> 4
- net CS24_h: track 0.00 -> 57.3 mm, vias 0 -> 2
- net CS22_neg_h: track 0.00 -> 57.0 mm, vias 0 -> 4
- net CS44_neg_h: track 0.00 -> 49.4 mm, vias 0 -> 6
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