File: analog_NN.kicad_pcb (KiCad board)
At the start: 4 copper layers, 230 parts, among them J1 Conn_01x01, J2 Conn_01x01, J3 Conn_01x01, J4 Conn_01x01, J7 Conn_01x01, U100 AD5160, U101 AD5160, U102 AD5160, U103 AD5160, U104 AD5160, U105 AD5160, U106 AD5160, U107 AD5160, U108 AD5160, U109 AD5160, U110 AD5160, U111 AD5160, U112 AD5160, U113 AD5160, U114 AD5160, U115 AD5160, U116 AD5160, U117 AD5160, U118 AD5160, U119 AD5160, U120 AD5160, U121 AD5160, U122 AD5160, U123 AD5160, U124 AD5160, U125 AD5160, U126 AD5160, U127 AD5160, U128 AD5160, U129 AD5160, U130 AD5160, U131 AD5160, U132 TLV9061xDBV, U28 AD5160, U29 AD5160, U30 AD5160, U31 AD5160, U32 AD5160, U33 AD5160, U34 AD5160, U35 AD5160, U36 74HC595, U37 74HC595, U38 74HC595, U39 74HC595, U43 TLV9061xDBV, U60 AD5160, U61 AD5160, U62 AD5160, U63 AD5160, U64 AD5160, U65 AD5160, U66 AD5160, U67 AD5160, U68 AD5160, U69 AD5160, U70 AD5160, U71 AD5160, U72 AD5160, U73 AD5160, U74 AD5160, U75 AD5160, U76 AD5160, U77 AD5160, U78 AD5160, U79 AD5160, U80 AD5160, U81 AD5160, U82 AD5160, U83 AD5160, U93 74HC595, U94 74HC595, U95 74HC595, U96 74HC595

Commit message: Updeated: pcb tracing
Parts:
- moved R33 88.8 mm to (174.5, 156.0), turned to 90 degrees
- moved R34 88.6 mm to (175.7, 159.8)
- moved R27 81.2 mm to (163.7, 143.1), turned to 90 degrees
- moved R32 77.9 mm to (164.2, 155.7), turned to 90 degrees
- moved U20 73.6 mm to (169.8, 155.5)
- moved R28 71.3 mm to (175.2, 142.6), turned to 90 degrees
- moved R29 71.0 mm to (176.3, 146.3)
- moved R47 70.8 mm to (193.8, 162.3), turned to 180 degrees
- moved R30 70.5 mm to (187.8, 155.2)
- moved R31 70.1 mm to (184.1, 156.3), turned to -90 degrees
- moved R22 65.3 mm to (163.9, 130.3), turned to 90 degrees
- moved U21 64.5 mm to (179.1, 156.0)
- moved U24 62.5 mm to (264.2, 149.1)
- moved U25 62.5 mm to (264.2, 153.7)
- moved U26 62.5 mm to (264.2, 158.4)
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Routing:
- net cbar1: track 182.7 -> 343.7 mm, vias 24 -> 28
- net VREF: track 746.2 -> 889.4 mm, vias 70 -> 93
- net cbar2: track 185.1 -> 322.2 mm, vias 24 -> 32
- net cbar4: track 146.9 -> 275.6 mm, vias 20 -> 32
- net cbar3: track 167.0 -> 277.8 mm, vias 22 -> 30
- net VDD: track 242.5 -> 310.0 mm, vias 0 -> 39
- net GND: track 216.7 -> 284.2 mm, vias 0 -> 39
- net Net-(U11-+): track 0.00 -> 25.5 mm
- net Net-(U15-+): track 0.00 -> 25.4 mm
- net Net-(U19-+): track 0.00 -> 24.6 mm
- net Net-(U23-+): track 0.00 -> 23.6 mm
- net Net-(U14--): track 0.00 -> 23.3 mm
- net Net-(U13-+): track 0.00 -> 22.8 mm, vias 0 -> 2
- net Net-(U17-+): track 0.00 -> 22.6 mm, vias 0 -> 2
- net Net-(U9-+): track 0.00 -> 22.2 mm, vias 0 -> 2
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Other:
- board text removed: "C5"
- board text removed: "C6"
- board text removed: "C7"
