File: crossbar_u.kicad_sch (KiCad schematic)
At the start: 48 parts, among them U60 AD5160, U61 AD5160, U62 AD5160, U63 AD5160, U64 AD5160, U65 AD5160, U66 AD5160, U67 AD5160, U68 AD5160, U69 AD5160, U70 AD5160, U71 AD5160, U72 AD5160, U73 AD5160, U74 AD5160, U75 AD5160, U76 AD5160, U77 AD5160, U78 AD5160, U79 AD5160, U80 AD5160, U81 AD5160, U82 AD5160, U83 AD5160

Commit message: updated capacitor values
Parts:
- C10, C11, C12, C13, C14, C15, C16, C17, C18, C19, C20, C21, C22, C23, C24, C25, C26, C27, C28, C5, C6, C7, C8, C9: value C -> 100nF
Changed lines of the file:
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@@
 			)
 		)
-		(property "Value" "C"
+		(property "Value" "100nF"
 			(at 35.56 214.6301 0)
 			(effects
@@
 			)
 		)
-		(property "Value" "C"
+		(property "Value" "100nF"
 			(at 111.76 147.3201 0)
 			(effects
@@
 			)
 		)
-		(property "Value" "C"
+		(property "Value" "100nF"
 			(at 177.8 124.4599 0)
 			(effects
@@
 			)
 		)
-		(property "Value" "C"
+		(property "Value" "100nF"
 			(at 73.66 214.6301 0)
 			(effects
@@
 			)
 		)
-		(property "Value" "C"
+		(property "Value" "100nF"
 			(at 177.8 191.7699 0)
 			(effects
@@
 			)
 		)
-		(property "Value" "C"
+		(property "Value" "100nF"
 			(at 63.5 124.4599 0)
 			(effects
@@
 			)
 		)
-		(property "Value" "C"
+		(property "Value" "100nF"
 			(at 101.6 57.1499 0)
 			(effects
@@
 			)
 		)
-		(property "Value" "C"
+		(property "Value" "100nF"
 			(at 73.66 80.0101 0)
 			(effects
@@
 			)
 		)
-		(property "Value" "C"
+		(property "Value" "100nF"
 			(at 111.76 80.0101 0)
 			(effects
@@
 			)
 		)
-		(property "Value" "C"
+		(property "Value" "100nF"
 			(at 149.86 147.3201 0)
 			(effects
@@
 			)
 		)
-		(property "Value" "C"
+		(property "Value" "100nF"
 			(at 139.7 57.1499 0)
 			(effects
@@
 			)
 		)
-		(property "Value" "C"
+		(property "Value" "100nF"
 			(at 101.6 191.7699 0)
 			(effects
@@
 			)
 		)
-		(property "Value" "C"
+		(property "Value" "100nF"
 			(at 111.76 214.6301 0)
 			(effects
@@
 			)
 		)
-		(property "Value" "C"
+		(property "Value" "100nF"
 			(at 63.5 57.1499 0)
 			(effects
@@
 			)
 		)
-		(property "Value" "C"
+		(property "Value" "100nF"
 			(at 149.86 214.6301 0)
 			(effects
@@
 			)
 		)
-		(property "Value" "C"
+		(property "Value" "100nF"
 			(at 35.56 80.0101 0)
 			(effects
@@
 			)
 		)
-		(property "Value" "C"
+		(property "Value" "100nF"
 			(at 149.86 80.0101 0)
 			(effects
@@
 			)
 		)
-		(property "Value" "C"
+		(property "Value" "100nF"
 			(at 73.66 147.3201 0)
 			(effects
@@
 			)
 		)
-		(property "Value" "C"
+		(property "Value" "100nF"
 			(at 139.7 124.4599 0)
 			(effects
@@
 			)
 		)
-		(property "Value" "C"
+		(property "Value" "100nF"
 			(at 177.8 57.1499 0)
 			(effects
@@
 			)
 		)
-		(property "Value" "C"
+		(property "Value" "100nF"
 			(at 63.5 191.7699 0)
 			(effects
@@
 			)
 		)
-		(property "Value" "C"
+		(property "Value" "100nF"
 			(at 101.6 124.4599 0)
 			(effects
@@
 			)
 		)
-		(property "Value" "C"
+		(property "Value" "100nF"
 			(at 35.56 147.3201 0)
 			(effects
@@
 			)
 		)
-		(property "Value" "C"
+		(property "Value" "100nF"
 			(at 139.7 191.7699 0)
 			(effects

Commit message: Updated: power
Other:
- moved on the sheet: C5

Commit message: Updated: op amps
Parts:
- C10, C11, C12, C13, C14, C15, C16, C17, C18, C19, C20, C21, C22, C23, C24, C25, C26, C27, C28, C5, C6, C7, C8, C9: footprint (none) -> Capacitor_SMD:C_1206_3216Metric_Pad1.33x1.80mm_HandSolder
Changed lines of the file:
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@@
 			)
 		)
-		(property "Footprint" ""
+		(property "Footprint" "Capacitor_SMD:C_1206_3216Metric_Pad1.33x1.80mm_HandSolder"
 			(at 174.9552 128.27 0)
 			(effects
@@
 			)
 		)
-		(property "Footprint" ""
+		(property "Footprint" "Capacitor_SMD:C_1206_3216Metric_Pad1.33x1.80mm_HandSolder"
 			(at 76.5048 76.2 0)
 			(effects
@@
 			)
 		)
-		(property "Footprint" ""
+		(property "Footprint" "Capacitor_SMD:C_1206_3216Metric_Pad1.33x1.80mm_HandSolder"
 			(at 98.7552 60.96 0)
 			(effects
@@
 			)
 		)
-		(property "Footprint" ""
+		(property "Footprint" "Capacitor_SMD:C_1206_3216Metric_Pad1.33x1.80mm_HandSolder"
 			(at 114.6048 143.51 0)
 			(effects
@@
 			)
 		)
-		(property "Footprint" ""
+		(property "Footprint" "Capacitor_SMD:C_1206_3216Metric_Pad1.33x1.80mm_HandSolder"
 			(at 38.4048 143.51 0)
 			(effects
@@
 			)
 		)
-		(property "Footprint" ""
+		(property "Footprint" "Capacitor_SMD:C_1206_3216Metric_Pad1.33x1.80mm_HandSolder"
 			(at 60.6552 195.58 0)
 			(effects
@@
 			)
 		)
-		(property "Footprint" ""
+		(property "Footprint" "Capacitor_SMD:C_1206_3216Metric_Pad1.33x1.80mm_HandSolder"
 			(at 136.8552 60.96 0)
 			(effects
@@
 			)
 		)
-		(property "Footprint" ""
+		(property "Footprint" "Capacitor_SMD:C_1206_3216Metric_Pad1.33x1.80mm_HandSolder"
 			(at 136.8552 195.58 0)
 			(effects
@@
 			)
 		)
-		(property "Footprint" ""
+		(property "Footprint" "Capacitor_SMD:C_1206_3216Metric_Pad1.33x1.80mm_HandSolder"
 			(at 114.6048 76.2 0)
 			(effects
@@
 			)
 		)
-		(property "Footprint" ""
+		(property "Footprint" "Capacitor_SMD:C_1206_3216Metric_Pad1.33x1.80mm_HandSolder"
 			(at 114.6048 210.82 0)
 			(effects
@@
 			)
 		)
-		(property "Footprint" ""
+		(property "Footprint" "Capacitor_SMD:C_1206_3216Metric_Pad1.33x1.80mm_HandSolder"
 			(at 38.4048 76.2 0)
 			(effects
@@
 			)
 		)
-		(property "Footprint" ""
+		(property "Footprint" "Capacitor_SMD:C_1206_3216Metric_Pad1.33x1.80mm_HandSolder"
 			(at 136.8552 128.27 0)
 			(effects
@@
 			)
 		)
-		(property "Footprint" ""
+		(property "Footprint" "Capacitor_SMD:C_1206_3216Metric_Pad1.33x1.80mm_HandSolder"
 			(at 38.4048 210.82 0)
 			(effects
@@
 			)
 		)
-		(property "Footprint" ""
+		(property "Footprint" "Capacitor_SMD:C_1206_3216Metric_Pad1.33x1.80mm_HandSolder"
 			(at 98.7552 128.27 0)
 			(effects
@@
 			)
 		)
-		(property "Footprint" ""
+		(property "Footprint" "Capacitor_SMD:C_1206_3216Metric_Pad1.33x1.80mm_HandSolder"
 			(at 174.9552 60.96 0)
 			(effects
@@
 			)
 		)
-		(property "Footprint" ""
+		(property "Footprint" "Capacitor_SMD:C_1206_3216Metric_Pad1.33x1.80mm_HandSolder"
 			(at 76.5048 210.82 0)
 			(effects
@@
 			)
 		)
-		(property "Footprint" ""
+		(property "Footprint" "Capacitor_SMD:C_1206_3216Metric_Pad1.33x1.80mm_HandSolder"
 			(at 152.7048 76.2 0)
 			(effects
@@
 			)
 		)
-		(property "Footprint" ""
+		(property "Footprint" "Capacitor_SMD:C_1206_3216Metric_Pad1.33x1.80mm_HandSolder"
 			(at 152.7048 143.51 0)
 			(effects
@@
 			)
 		)
-		(property "Footprint" ""
+		(property "Footprint" "Capacitor_SMD:C_1206_3216Metric_Pad1.33x1.80mm_HandSolder"
 			(at 60.6552 60.96 0)
 			(effects
@@
 			)
 		)
-		(property "Footprint" ""
+		(property "Footprint" "Capacitor_SMD:C_1206_3216Metric_Pad1.33x1.80mm_HandSolder"
 			(at 152.7048 210.82 0)
 			(effects
@@
 			)
 		)
-		(property "Footprint" ""
+		(property "Footprint" "Capacitor_SMD:C_1206_3216Metric_Pad1.33x1.80mm_HandSolder"
 			(at 60.6552 128.27 0)
 			(effects
@@
 			)
 		)
-		(property "Footprint" ""
+		(property "Footprint" "Capacitor_SMD:C_1206_3216Metric_Pad1.33x1.80mm_HandSolder"
 			(at 98.7552 195.58 0)
 			(effects
@@
 			)
 		)
-		(property "Footprint" ""
+		(property "Footprint" "Capacitor_SMD:C_1206_3216Metric_Pad1.33x1.80mm_HandSolder"
 			(at 76.5048 143.51 0)
 			(effects
@@
 			)
 		)
-		(property "Footprint" ""
+		(property "Footprint" "Capacitor_SMD:C_1206_3216Metric_Pad1.33x1.80mm_HandSolder"
 			(at 174.9552 195.58 0)
 			(effects

Commit message: Updated: pots
Connections:
- net CLK: now also U80.4 (CLK), U81.4 (CLK), U82.4 (CLK), U83.4 (CLK)
- net SDI: now also U80.5 (SDI), U81.5 (SDI), U82.5 (SDI), U83.5 (SDI)
- net cbar1: now also U64.8 (A), U72.8 (A), U80.8 (A); no longer U64.7 (B), U72.7 (B), U80.7 (B)
- net cbar2: now also U65.8 (A), U73.8 (A), U81.8 (A); no longer U65.7 (B), U73.7 (B), U81.7 (B)
- net cbar3: now also U66.8 (A), U74.8 (A), U82.8 (A); no longer U66.7 (B), U74.7 (B), U82.7 (B)
- net cbar4: now also U67.8 (A), U75.8 (A), U83.8 (A); no longer U67.7 (B), U75.7 (B), U83.7 (B)
- net VREF: now reaches U61.7 (B)
- net VREF: now also U60.7 (B), U62.7 (B), U63.7 (B), U64.7 (B), U65.7 (B), U66.7 (B), U67.7 (B), U68.7 (B), U69.7 (B), U70.7 (B), U71.7 (B), U72.7 (B), U73.7 (B), U74.7 (B), U75.7 (B), U76.7 (B), U77.7 (B), U78.7 (B), U79.7 (B), U80.7 (B), U81.7 (B), U82.7 (B), U83.7 (B)

Commit message: Updated: crossbar
Parts:
- C10, C11, C12, C13, C14, C15, C16, C17, C18, C19, C20, C21, C22, C23, C24, C25, C26, C27, C28, C5, C6, C7, C8, C9: footprint Capacitor_SMD:C_1206_3216Metric_Pad1.33x1.80mm_HandSolder -> Capacitor_SMD:C_1206_3216Metric
Changed lines of the file:
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@@
 	)
 	(junction
+		(at 35.56 52.07)
+		(diameter 0)
+		(color 0 0 0 0)
+	)
+	(junction
 		(at 163.83 97.79)
 		(diameter 0)
@@
 	(wire
 		(pts
+			(xy 35.56 52.07) (xy 39.37 52.07)
+		)
+		(stroke
+			(width 0)
+			(type default)
+		)
+	)
+	(wire
+		(pts
 			(xy 163.83 173.99) (xy 163.83 176.53)
 		)
@@
 	(wire
 		(pts
+			(xy 33.02 52.07) (xy 35.56 52.07)
+		)
+		(stroke
+			(width 0)
+			(type default)
+		)
+	)
+	(wire
+		(pts
 			(xy 69.85 132.08) (xy 69.85 134.62)
 		)
@@
 			)
 		)
-		(property "Footprint" "Capacitor_SMD:C_1206_3216Metric_Pad1.33x1.80mm_HandSolder"
+		(property "Footprint" "Capacitor_SMD:C_1206_3216Metric"
 			(at 174.9552 128.27 0)
 			(effects
@@
 			)
 		)
-		(property "Footprint" "Capacitor_SMD:C_1206_3216Metric_Pad1.33x1.80mm_HandSolder"
+		(property "Footprint" "Capacitor_SMD:C_1206_3216Metric"
 			(at 76.5048 76.2 0)
 			(effects
@@
 			)
 		)
-		(property "Footprint" "Capacitor_SMD:C_1206_3216Metric_Pad1.33x1.80mm_HandSolder"
+		(property "Footprint" "Capacitor_SMD:C_1206_3216Metric"
 			(at 98.7552 60.96 0)
 			(effects
@@
 			)
 		)
-		(property "Footprint" "Capacitor_SMD:C_1206_3216Metric_Pad1.33x1.80mm_HandSolder"
+		(property "Footprint" "Capacitor_SMD:C_1206_3216Metric"
 			(at 114.6048 143.51 0)
 			(effects
@@
 			)
 		)
-		(property "Footprint" "Capacitor_SMD:C_1206_3216Metric_Pad1.33x1.80mm_HandSolder"
+		(property "Footprint" "Capacitor_SMD:C_1206_3216Metric"
 			(at 38.4048 143.51 0)
 			(effects
@@
 			)
 		)
-		(property "Footprint" "Capacitor_SMD:C_1206_3216Metric_Pad1.33x1.80mm_HandSolder"
+		(property "Footprint" "Capacitor_SMD:C_1206_3216Metric"
 			(at 60.6552 195.58 0)
 			(effects
@@
 			)
 		)
-		(property "Footprint" "Capacitor_SMD:C_1206_3216Metric_Pad1.33x1.80mm_HandSolder"
+		(property "Footprint" "Capacitor_SMD:C_1206_3216Metric"
 			(at 136.8552 60.96 0)
 			(effects
@@
 			)
 		)
-		(property "Footprint" "Capacitor_SMD:C_1206_3216Metric_Pad1.33x1.80mm_HandSolder"
+		(property "Footprint" "Capacitor_SMD:C_1206_3216Metric"
 			(at 136.8552 195.58 0)
 			(effects
@@
 			)
 		)
-		(property "Footprint" "Capacitor_SMD:C_1206_3216Metric_Pad1.33x1.80mm_HandSolder"
+		(property "Footprint" "Capacitor_SMD:C_1206_3216Metric"
 			(at 114.6048 76.2 0)
 			(effects
@@
 			)
 		)
-		(property "Footprint" "Capacitor_SMD:C_1206_3216Metric_Pad1.33x1.80mm_HandSolder"
+		(property "Footprint" "Capacitor_SMD:C_1206_3216Metric"
 			(at 114.6048 210.82 0)
 			(effects
@@
 			)
 		)
-		(property "Footprint" "Capacitor_SMD:C_1206_3216Metric_Pad1.33x1.80mm_HandSolder"
+		(property "Footprint" "Capacitor_SMD:C_1206_3216Metric"
 			(at 38.4048 76.2 0)
 			(effects
@@
 			)
 		)
-		(property "Footprint" "Capacitor_SMD:C_1206_3216Metric_Pad1.33x1.80mm_HandSolder"
+		(property "Footprint" "Capacitor_SMD:C_1206_3216Metric"
 			(at 136.8552 128.27 0)
 			(effects
@@
 			)
 		)
-		(property "Footprint" "Capacitor_SMD:C_1206_3216Metric_Pad1.33x1.80mm_HandSolder"
+		(property "Footprint" "Capacitor_SMD:C_1206_3216Metric"
 			(at 38.4048 210.82 0)
 			(effects
@@
 			)
 		)
-		(property "Footprint" "Capacitor_SMD:C_1206_3216Metric_Pad1.33x1.80mm_HandSolder"
+		(property "Footprint" "Capacitor_SMD:C_1206_3216Metric"
 			(at 98.7552 128.27 0)
 			(effects
@@
 			)
 		)
-		(property "Footprint" "Capacitor_SMD:C_1206_3216Metric_Pad1.33x1.80mm_HandSolder"
+		(property "Footprint" "Capacitor_SMD:C_1206_3216Metric"
 			(at 174.9552 60.96 0)
 			(effects
@@
 			)
 		)
-		(property "Footprint" "Capacitor_SMD:C_1206_3216Metric_Pad1.33x1.80mm_HandSolder"
+		(property "Footprint" "Capacitor_SMD:C_1206_3216Metric"
 			(at 76.5048 210.82 0)
 			(effects
@@
 			)
 		)
-		(property "Footprint" "Capacitor_SMD:C_1206_3216Metric_Pad1.33x1.80mm_HandSolder"
+		(property "Footprint" "Capacitor_SMD:C_1206_3216Metric"
 			(at 152.7048 76.2 0)
 			(effects
@@
 			)
 		)
-		(property "Footprint" "Capacitor_SMD:C_1206_3216Metric_Pad1.33x1.80mm_HandSolder"
+		(property "Footprint" "Capacitor_SMD:C_1206_3216Metric"
 			(at 152.7048 143.51 0)
 			(effects
@@
 			)
 		)
-		(property "Footprint" "Capacitor_SMD:C_1206_3216Metric_Pad1.33x1.80mm_HandSolder"
+		(property "Footprint" "Capacitor_SMD:C_1206_3216Metric"
 			(at 60.6552 60.96 0)
 			(effects
@@
 	)
 	(symbol
+		(lib_id "power:PWR_FLAG")
+		(at 35.56 52.07 0)
+		(unit 1)
+		(exclude_from_sim no)
+		(in_bom yes)
+		(on_board yes)
+		(dnp no)
+		(fields_autoplaced yes)
+		(property "Reference" "#FLG03"
+			(at 35.56 50.165 0)
+			(effects
+				(font
+					(size 1.27 1.27)
+				)
+				(hide yes)
+			)
+		)
+		(property "Value" "PWR_FLAG"
+			(at 35.56 46.99 0)
+			(effects
+				(font
+					(size 1.27 1.27)
+				)
+			)
+		)
+		(property "Footprint" ""
+			(at 35.56 52.07 0)
+			(effects
+				(font
+					(size 1.27 1.27)
+				)
+				(hide yes)
+			)
+		)
+		(property "Datasheet" "~"
+			(at 35.56 52.07 0)
+			(effects
+				(font
+					(size 1.27 1.27)
+				)
+				(hide yes)
+			)
+		)
+		(property "Description" "Special symbol for telling ERC where power comes from"
+			(at 35.56 52.07 0)
+			(effects
+				(font
+					(size 1.27 1.27)
+				)
+				(hide yes)
+			)
+		)
+		(pin "1"
+		)
+		(instances
+			(project ""
+				(path "/8de080c9-ac72-4350-b5d3-2d90d26f0ccc/be605785-53c8-4b82-8661-40dd21e1d9cd/266ed6db-bf88-40c2-a324-1d8d44147eb4"
+					(reference "#FLG03")
+					(unit 1)
+				)
+			)
+		)
+	)
+	(symbol
 		(lib_id "Device:C")
 		(at 153.67 214.63 180)
@@
 			)
 		)
-		(property "Footprint" "Capacitor_SMD:C_1206_3216Metric_Pad1.33x1.80mm_HandSolder"
+		(property "Footprint" "Capacitor_SMD:C_1206_3216Metric"
 			(at 152.7048 210.82 0)
 			(effects
@@
 			)
 		)
-		(property "Footprint" "Capacitor_SMD:C_1206_3216Metric_Pad1.33x1.80mm_HandSolder"
+		(property "Footprint" "Capacitor_SMD:C_1206_3216Metric"
 			(at 60.6552 128.27 0)
 			(effects
@@
 			)
 		)
-		(property "Footprint" "Capacitor_SMD:C_1206_3216Metric_Pad1.33x1.80mm_HandSolder"
+		(property "Footprint" "Capacitor_SMD:C_1206_3216Metric"
 			(at 98.7552 195.58 0)
 			(effects
@@
 			)
 		)
-		(property "Footprint" "Capacitor_SMD:C_1206_3216Metric_Pad1.33x1.80mm_HandSolder"
+		(property "Footprint" "Capacitor_SMD:C_1206_3216Metric"
 			(at 76.5048 143.51 0)
 			(effects
@@
 	(symbol
 		(lib_id "power:GND")
-		(at 39.37 52.07 270)
+		(at 33.02 52.07 270)
 		(unit 1)
 		(exclude_from_sim no)
@@
 		(fields_autoplaced yes)
 		(property "Reference" "#PWR031"
-			(at 33.02 52.07 0)
+			(at 26.67 52.07 0)
 			(effects
 				(font
@@
 		)
 		(property "Value" "GND"
-			(at 35.56 52.0699 90)
+			(at 29.21 52.0699 90)
 			(effects
 				(font
@@
 		)
 		(property "Footprint" ""
-			(at 39.37 52.07 0)
+			(at 33.02 52.07 0)
 			(effects
 				(font
@@
 		)
 		(property "Datasheet" ""
-			(at 39.37 52.07 0)
+			(at 33.02 52.07 0)
 			(effects
 				(font
@@
 		)
 		(property "Description" "Power symbol creates a global label with name \"GND\" , ground"
-			(at 39.37 52.07 0)
+			(at 33.02 52.07 0)
 			(effects
 				(font
@@
 			)
 		)
-		(property "Footprint" "Capacitor_SMD:C_1206_3216Metric_Pad1.33x1.80mm_HandSolder"
+		(property "Footprint" "Capacitor_SMD:C_1206_3216Metric"
 			(at 174.9552 195.58 0)
 			(effects
