File: _autosave-analog_NN.kicad_pcb (KiCad board)
At the start: 4 copper layers, 230 parts, among them J1 Conn_01x01, J2 Conn_01x01, J3 Conn_01x01, J4 Conn_01x01, J5 Conn_01x01, J6 Conn_01x01, J7 Conn_01x01, U100 AD5160, U101 AD5160, U102 AD5160, U103 AD5160, U104 AD5160, U105 AD5160, U106 AD5160, U107 AD5160, U108 AD5160, U109 AD5160, U110 AD5160, U111 AD5160, U112 AD5160, U113 AD5160, U114 AD5160, U115 AD5160, U116 AD5160, U117 AD5160, U118 AD5160, U119 AD5160, U120 AD5160, U121 AD5160, U122 AD5160, U123 AD5160, U124 AD5160, U125 AD5160, U126 AD5160, U127 AD5160, U128 AD5160, U129 AD5160, U130 AD5160, U131 AD5160, U132 TLV9061xDBV, U28 AD5160, U29 AD5160, U30 AD5160, U31 AD5160, U32 AD5160, U33 AD5160, U34 AD5160, U35 AD5160, U36 74HC595, U37 74HC595, U38 74HC595, U39 74HC595, U43 TLV9061xDBV, U60 AD5160, U61 AD5160, U62 AD5160, U63 AD5160, U64 AD5160, U65 AD5160, U66 AD5160, U67 AD5160, U68 AD5160, U69 AD5160, U70 AD5160, U71 AD5160, U72 AD5160, U73 AD5160, U74 AD5160, U75 AD5160, U76 AD5160, U77 AD5160, U78 AD5160, U79 AD5160, U80 AD5160, U81 AD5160, U82 AD5160, U83 AD5160, U93 74HC595, U94 74HC595, U95 74HC595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

Commit message: Updated: sim folder
Parts:
- moved R14 257.4 mm to (32.1, 122.0), turned to 180 degrees
- moved R12 256.5 mm to (32.0, 105.4), turned to 180 degrees
- moved R8 250.7 mm to (31.4, 77.8), turned to 180 degrees
- moved R13 250.6 mm to (38.8, 117.2), turned to 180 degrees
- moved R10 249.9 mm to (32.0, 91.4), turned to 180 degrees
- moved R11 249.3 mm to (39.1, 101.3), turned to 180 degrees
- moved R7 243.2 mm to (38.9, 74.2), turned to 180 degrees
- moved R9 242.9 mm to (39.1, 87.6), turned to 180 degrees
- moved U7 234.5 mm to (39.3, 121.9), turned to 180 degrees
- moved U6 233.2 mm to (39.1, 106.1), turned to 180 degrees
- moved U4 227.3 mm to (38.8, 78.8), turned to 180 degrees
- moved U5 226.8 mm to (39.0, 92.2), turned to 180 degrees
- moved C12 201.5 mm to (79.2, 42.4)
- moved C5 199.8 mm to (76.2, 25.4), turned to 90 degrees
- moved C6 185.2 mm to (91.3, 25.1), turned to 90 degrees
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Routing:
- net VDD: track 3.10 -> 23.7 mm, vias 2 -> 7
- net GND: track 3.07 -> 22.2 mm, vias 2 -> 10
- net Net-(U3--): track 0.00 -> 9.92 mm
- net -Vu3: track 0.00 -> 9.67 mm
- net Net-(U7--): track 0.00 -> 9.13 mm
- net Net-(U4--): track 0.00 -> 8.62 mm
- net Net-(U6--): track 0.00 -> 8.59 mm
- net -Vh4: track 0.00 -> 8.42 mm
- net -Vh3: track 0.00 -> 8.34 mm
- net -Vh2: track 0.00 -> 8.33 mm
- net Net-(U5--): track 0.00 -> 8.14 mm
- net VREF: track 3.10 -> 10.7 mm, vias 2 -> 7
- net Vu3: track 0.00 -> 6.14 mm
