File: _autosave-analog_NN.kicad_pcb (KiCad board)
At the start: 4 copper layers, 230 parts, among them J1 Conn_01x01, J2 Conn_01x01, J3 Conn_01x01, J4 Conn_01x01, J7 Conn_01x01, U100 AD5160, U101 AD5160, U102 AD5160, U103 AD5160, U104 AD5160, U105 AD5160, U106 AD5160, U107 AD5160, U108 AD5160, U109 AD5160, U110 AD5160, U111 AD5160, U112 AD5160, U113 AD5160, U114 AD5160, U115 AD5160, U116 AD5160, U117 AD5160, U118 AD5160, U119 AD5160, U120 AD5160, U121 AD5160, U122 AD5160, U123 AD5160, U124 AD5160, U125 AD5160, U126 AD5160, U127 AD5160, U128 AD5160, U129 AD5160, U130 AD5160, U131 AD5160, U132 TLV9061xDBV, U28 AD5160, U29 AD5160, U30 AD5160, U31 AD5160, U32 AD5160, U33 AD5160, U34 AD5160, U35 AD5160, U36 74HC595, U37 74HC595, U38 74HC595, U39 74HC595, U43 TLV9061xDBV, U60 AD5160, U61 AD5160, U62 AD5160, U63 AD5160, U64 AD5160, U65 AD5160, U66 AD5160, U67 AD5160, U68 AD5160, U69 AD5160, U70 AD5160, U71 AD5160, U72 AD5160, U73 AD5160, U74 AD5160, U75 AD5160, U76 AD5160, U77 AD5160, U78 AD5160, U79 AD5160, U80 AD5160, U81 AD5160, U82 AD5160, U83 AD5160, U93 74HC595, U94 74HC595, U95 74HC595, U96 74HC595

Commit message: Updated: pcb
Parts:
- moved U11 90.0 mm to (237.2, 31.2)
- moved U10 83.4 mm to (230.3, 31.1)
- moved U12 83.1 mm to (263.6, 38.4)
- moved U13 83.1 mm to (263.6, 43.0)
- moved U14 83.1 mm to (263.6, 47.6)
- moved U15 83.1 mm to (263.6, 52.2)
- moved C2 83.1 mm to (279.3, 41.0)
- moved C3 83.1 mm to (279.3, 44.4)
- moved C4 83.1 mm to (279.3, 47.7)
- moved R17 83.1 mm to (258.7, 24.4)
- moved R20 83.1 mm to (258.7, 34.3)
- moved R21 83.1 mm to (264.3, 17.8)
- moved R22 83.1 mm to (264.3, 21.1)
- moved R23 83.1 mm to (264.3, 24.4)
- moved R24 83.1 mm to (264.3, 27.7)
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Routing:
- net GND: track 216.7 -> 265.5 mm, vias 0 -> 27
- net VDD: track 242.5 -> 290.9 mm, vias 0 -> 27
- net VREF: track 746.2 -> 788.6 mm, vias 70 -> 80
- net Net-(U11-+): track 0.00 -> 25.5 mm
- net Net-(U9-+): track 0.00 -> 22.2 mm, vias 0 -> 2
- net Net-(U10--): track 0.00 -> 21.5 mm
- net Net-(R16-Pad2): track 0.00 -> 13.1 mm
- net Vh1: track 0.00 -> 11.5 mm
- net -Vh1: track 52.1 -> 60.5 mm
- net cbar1: track 182.7 -> 190.2 mm
- net Net-(U9--): track 0.00 -> 6.42 mm
- net CS42_neg: track 28.7 -> 29.6 mm
Other:
- board text removed: "C5"
- board text removed: "C6"
- board text removed: "C7"
