File: shift_register_chain.kicad_sch (KiCad schematic)
At the start: 8 parts, among them U36 74HC595, U37 74HC595, U38 74HC595, U39 74HC595, U93 74HC595, U94 74HC595, U95 74HC595, U96 74HC595

Commit message: Updated: power
Connections:
- net GND: now also U36.13 (~{OE}), U37.13 (~{OE}), U38.13 (~{OE}), U39.13 (~{OE}), U93.13 (~{OE}), U94.13 (~{OE}), U95.13 (~{OE}), U96.13 (~{OE})
- net VCC: now reaches U36.10 (~{SRCLR})
- net VCC: now also U36.16 (VCC), U37.10 (~{SRCLR}), U37.16 (VCC), U38.10 (~{SRCLR}), U38.16 (VCC), U39.10 (~{SRCLR}), U39.16 (VCC), U93.10 (~{SRCLR}), U93.16 (VCC), U94.10 (~{SRCLR}), U94.16 (VCC), U95.10 (~{SRCLR}), U95.16 (VCC), U96.10 (~{SRCLR}), U96.16 (VCC)
- net SRCLK: now reaches U36.11 (SRCLK)
- net SRCLK: now also U37.11 (SRCLK), U38.11 (SRCLK), U39.11 (SRCLK), U93.11 (SRCLK), U94.11 (SRCLK), U95.11 (SRCLK), U96.11 (SRCLK)
- net RCLK: now reaches U36.12 (RCLK)
- net RCLK: now also U37.12 (RCLK), U38.12 (RCLK), U39.12 (RCLK), U93.12 (RCLK), U94.12 (RCLK), U95.12 (RCLK), U96.12 (RCLK)
- net ser: now reaches U93.14 (SER)

Commit message: Updated: crossbar
Parts:
- U36, U37, U38, U39, U93, U94, U95, U96: footprint (none) -> Package_SO:SOIC-16_3.9x9.9mm_P1.27mm
Connections:
- net VCC: no longer U36.10 (~{SRCLR}), U36.16 (VCC), U37.16 (VCC), U38.16 (VCC), U39.16 (VCC), U93.16 (VCC), U94.16 (VCC), U95.16 (VCC), U96.16 (VCC)
- new net VDD: U36.10 (~{SRCLR}), U36.16 (VCC), U37.16 (VCC), U38.16 (VCC), U39.16 (VCC), U93.16 (VCC), U94.16 (VCC), U95.16 (VCC), U96.16 (VCC)
- no-connect marks 0 -> 1
Changed lines of the file:
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@@
 	(generator_version "9.0")
 	(paper "A4")
+	(junction
+		(at 102.87 107.95)
+		(diameter 0)
+		(color 0 0 0 0)
+	)
+	(no_connect
+		(at 248.92 123.19)
+	)
 	(wire
 		(pts
@@
 	(wire
 		(pts
+			(xy 102.87 107.95) (xy 109.22 107.95)
+		)
+		(stroke
+			(width 0)
+			(type default)
+		)
+	)
+	(wire
+		(pts
 			(xy 151.13 100.33) (xy 151.13 123.19)
 		)
@@
 	(wire
 		(pts
+			(xy 99.06 107.95) (xy 102.87 107.95)
+		)
+		(stroke
+			(width 0)
+			(type default)
+		)
+	)
+	(wire
+		(pts
 			(xy 212.09 35.56) (xy 229.87 35.56)
 		)
@@
 		)
 	)
-	(global_label "VCC"
+	(global_label "VDD"
 		(shape input)
 		(at 119.38 95.25 90)
@@
 		)
 	)
-	(global_label "VCC"
+	(global_label "VDD"
 		(shape input)
 		(at 120.65 30.48 90)
@@
 		)
 	)
-	(global_label "VCC"
+	(global_label "VDD"
 		(shape input)
 		(at 179.07 95.25 90)
@@
 		)
 	)
-	(global_label "VCC"
+	(global_label "VDD"
 		(shape input)
 		(at 60.96 30.48 90)
@@
 		)
 	)
-	(global_label "VCC"
+	(global_label "VDD"
 		(shape input)
 		(at 59.69 95.25 90)
@@
 	(global_label "VCC"
 		(shape input)
-		(at 109.22 107.95 180)
+		(at 99.06 107.95 180)
 		(fields_autoplaced yes)
 		(effects
@@
 		)
 		(property "Intersheetrefs" "${INTERSHEET_REFS}"
-			(at 102.6062 107.95 0)
+			(at 92.4462 107.95 0)
 			(effects
 				(font
@@
 		)
 	)
-	(global_label "VCC"
+	(global_label "VDD"
 		(shape input)
 		(at 49.53 107.95 180)
@@
 		)
 	)
-	(global_label "VCC"
+	(global_label "VDD"
 		(shape input)
 		(at 238.76 95.25 90)
@@
 		)
 	)
-	(global_label "VCC"
+	(global_label "VDD"
 		(shape input)
 		(at 180.34 30.48 90)
@@
 		)
 	)
-	(global_label "VCC"
+	(global_label "VDD"
 		(shape input)
 		(at 240.03 30.48 90)
@@
 			)
 		)
-		(property "Footprint" ""
+		(property "Footprint" "Package_SO:SOIC-16_3.9x9.9mm_P1.27mm"
 			(at 59.69 110.49 0)
 			(effects
@@
 			)
 		)
-		(property "Footprint" ""
+		(property "Footprint" "Package_SO:SOIC-16_3.9x9.9mm_P1.27mm"
 			(at 60.96 45.72 0)
 			(effects
@@
 	)
 	(symbol
+		(lib_id "power:PWR_FLAG")
+		(at 102.87 107.95 180)
+		(unit 1)
+		(exclude_from_sim no)
+		(in_bom yes)
+		(on_board yes)
+		(dnp no)
+		(property "Reference" "#FLG02"
+			(at 102.87 109.855 0)
+			(effects
+				(font
+					(size 1.27 1.27)
+				)
+				(hide yes)
+			)
+		)
+		(property "Value" "PWR_FLAG"
+			(at 97.79 110.744 0)
+			(effects
+				(font
+					(size 1.27 1.27)
+				)
+			)
+		)
+		(property "Footprint" ""
+			(at 102.87 107.95 0)
+			(effects
+				(font
+					(size 1.27 1.27)
+				)
+				(hide yes)
+			)
+		)
+		(property "Datasheet" "~"
+			(at 102.87 107.95 0)
+			(effects
+				(font
+					(size 1.27 1.27)
+				)
+				(hide yes)
+			)
+		)
+		(property "Description" "Special symbol for telling ERC where power comes from"
+			(at 102.87 107.95 0)
+			(effects
+				(font
+					(size 1.27 1.27)
+				)
+				(hide yes)
+			)
+		)
+		(pin "1"
+		)
+		(instances
+			(project ""
+				(path "/8de080c9-ac72-4350-b5d3-2d90d26f0ccc/702edd85-3e4b-44ec-b58a-808e908b41df"
+					(reference "#FLG02")
+					(unit 1)
+				)
+			)
+		)
+	)
+	(symbol
 		(lib_id "74xx:74HC595")
 		(at 119.38 110.49 0)
@@
 			)
 		)
-		(property "Footprint" ""
+		(property "Footprint" "Package_SO:SOIC-16_3.9x9.9mm_P1.27mm"
 			(at 119.38 110.49 0)
 			(effects
@@
 			)
 		)
-		(property "Footprint" ""
+		(property "Footprint" "Package_SO:SOIC-16_3.9x9.9mm_P1.27mm"
 			(at 179.07 110.49 0)
 			(effects
@@
 			)
 		)
-		(property "Footprint" ""
+		(property "Footprint" "Package_SO:SOIC-16_3.9x9.9mm_P1.27mm"
 			(at 120.65 45.72 0)
 			(effects
@@
 			)
 		)
-		(property "Footprint" ""
+		(property "Footprint" "Package_SO:SOIC-16_3.9x9.9mm_P1.27mm"
 			(at 238.76 110.49 0)
 			(effects
@@
 			)
 		)
-		(property "Footprint" ""
+		(property "Footprint" "Package_SO:SOIC-16_3.9x9.9mm_P1.27mm"
 			(at 240.03 45.72 0)
 			(effects
@@
 			)
 		)
-		(property "Footprint" ""
+		(property "Footprint" "Package_SO:SOIC-16_3.9x9.9mm_P1.27mm"
 			(at 180.34 45.72 0)
 			(effects

Commit message: Updated: schematic
Connections:
- net VCC is gone; now on net VDD: U37.10 (~{SRCLR}), U38.10 (~{SRCLR}), U39.10 (~{SRCLR}), U93.10 (~{SRCLR}), U94.10 (~{SRCLR}), U95.10 (~{SRCLR}), U96.10 (~{SRCLR})
Changed lines of the file:
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@@
 	(generator_version "9.0")
 	(paper "A4")
-	(junction
-		(at 102.87 107.95)
-		(diameter 0)
-		(color 0 0 0 0)
-	)
 	(no_connect
 		(at 248.92 123.19)
@@
 	(wire
 		(pts
-			(xy 102.87 107.95) (xy 109.22 107.95)
-		)
-		(stroke
-			(width 0)
-			(type default)
-		)
-	)
-	(wire
-		(pts
 			(xy 151.13 100.33) (xy 151.13 123.19)
 		)
@@
 	(wire
 		(pts
-			(xy 99.06 107.95) (xy 102.87 107.95)
+			(xy 99.06 107.95) (xy 109.22 107.95)
 		)
 		(stroke
@@
 		)
 	)
-	(global_label "VCC"
+	(global_label "VDD"
 		(shape input)
 		(at 168.91 107.95 180)
@@
 		)
 	)
-	(global_label "VCC"
+	(global_label "VDD"
 		(shape input)
 		(at 228.6 107.95 180)
@@
 		)
 	)
-	(global_label "VCC"
+	(global_label "VDD"
 		(shape input)
 		(at 170.18 43.18 180)
@@
 		)
 	)
-	(global_label "VCC"
+	(global_label "VDD"
 		(shape input)
 		(at 110.49 43.18 180)
@@
 		)
 	)
-	(global_label "VCC"
+	(global_label "VDD"
 		(shape input)
 		(at 99.06 107.95 180)
@@
 		)
 	)
-	(global_label "VCC"
+	(global_label "VDD"
 		(shape input)
 		(at 229.87 43.18 180)
@@
 		)
 	)
-	(global_label "VCC"
+	(global_label "VDD"
 		(shape input)
 		(at 50.8 43.18 180)
@@
 					(unit 1)
 				)
-			)
-		)
-	)
-	(symbol
-		(lib_id "power:PWR_FLAG")
-		(at 102.87 107.95 180)
-		(unit 1)
-		(exclude_from_sim no)
-		(in_bom yes)
-		(on_board yes)
-		(dnp no)
-		(property "Reference" "#FLG02"
-			(at 102.87 109.855 0)
-			(effects
-				(font
-					(size 1.27 1.27)
-				)
-				(hide yes)
-			)
-		)
-		(property "Value" "PWR_FLAG"
-			(at 97.79 110.744 0)
-			(effects
-				(font
-					(size 1.27 1.27)
-				)
-			)
-		)
-		(property "Footprint" ""
-			(at 102.87 107.95 0)
-			(effects
-				(font
-					(size 1.27 1.27)
-				)
-				(hide yes)
-			)
-		)
-		(property "Datasheet" "~"
-			(at 102.87 107.95 0)
-			(effects
-				(font
-					(size 1.27 1.27)
-				)
-				(hide yes)
-			)
-		)
-		(property "Description" "Special symbol for telling ERC where power comes from"
-			(at 102.87 107.95 0)
-			(effects
-				(font
-					(size 1.27 1.27)
-				)
-				(hide yes)
-			)
-		)
-		(pin "1"
-		)
-		(instances
-			(project ""
-				(path "/8de080c9-ac72-4350-b5d3-2d90d26f0ccc/702edd85-3e4b-44ec-b58a-808e908b41df"
-					(reference "#FLG02")
-					(unit 1)
-				)
