File: torque.kicad_sch (KiCad schematic)
At the start: 30 parts, among them U24 ${SIM.PARAMS}, U25 ${SIM.PARAMS}, U26 ${SIM.PARAMS}, U27 ${SIM.PARAMS}, U28 AD5160, U29 AD5160, U30 AD5160, U31 AD5160, U32 AD5160, U33 AD5160, U34 AD5160, U35 AD5160, U92 ${SIM.PARAMS}

Commit message: Updated: crossbar
Parts:
- added J7: Conn_01x01, analog_NN:WireSolderPad_1.0mm, symbol Connector_Generic:Conn_01x01
- C61, C62, C63, C64, C65, C66, C67, C68: footprint Capacitor_SMD:C_1206_3216Metric_Pad1.33x1.80mm_HandSolder -> Capacitor_SMD:C_1206_3216Metric
- R35, R36, R37, R38, R39, R40, R41, R42, R43: footprint Resistor_SMD:R_1206_3216Metric_Pad1.30x1.75mm_HandSolder -> Resistor_SMD:R_1206_3216Metric
Connections:
- net VCC is gone; now on net VDD: U24.5 (V+), U25.5 (V+), U26.5 (V+), U27.5 (V+), U92.5 (V+)
- net torque: now also J7.1 (Pin_1)
Changed lines of the file:
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@@
 		)
 	)
-	(global_label "VCC"
+	(global_label "VDD"
 		(shape input)
 		(at 107.95 205.74 90)
@@
 		)
 	)
-	(global_label "VCC"
+	(global_label "VDD"
 		(shape input)
 		(at 107.95 162.56 90)
@@
 		)
 	)
-	(global_label "VCC"
+	(global_label "VDD"
 		(shape input)
 		(at 107.95 119.38 90)
@@
 		)
 	)
+	(global_label "torque"
+		(shape input)
+		(at 250.19 179.07 180)
+		(fields_autoplaced yes)
+		(effects
+			(font
+				(size 1.27 1.27)
+			)
+			(justify right)
+		)
+		(property "Intersheetrefs" "${INTERSHEET_REFS}"
+			(at 241.1573 179.07 0)
+			(effects
+				(font
+					(size 1.27 1.27)
+				)
+				(justify right)
+				(hide yes)
+			)
+		)
+	)
 	(global_label "Wo4_neg"
 		(shape input)
@@
 		)
 	)
-	(global_label "VCC"
+	(global_label "VDD"
 		(shape input)
 		(at 214.63 171.45 90)
@@
 		)
 	)
-	(global_label "VCC"
+	(global_label "VDD"
 		(shape input)
 		(at 107.95 251.46 90)
@@
 			)
 		)
-		(property "Footprint" "Capacitor_SMD:C_1206_3216Metric_Pad1.33x1.80mm_HandSolder"
+		(property "Footprint" "Capacitor_SMD:C_1206_3216Metric"
 			(at 187.6552 83.82 0)
 			(effects
@@
 			)
 		)
-		(property "Footprint" "Resistor_SMD:R_1206_3216Metric_Pad1.30x1.75mm_HandSolder"
+		(property "Footprint" "Resistor_SMD:R_1206_3216Metric"
 			(at 215.9 198.628 90)
 			(effects
@@
 			)
 		)
-		(property "Footprint" "Resistor_SMD:R_1206_3216Metric_Pad1.30x1.75mm_HandSolder"
+		(property "Footprint" "Resistor_SMD:R_1206_3216Metric"
 			(at 110.49 195.072 90)
 			(effects
@@
 			)
 		)
-		(property "Footprint" "Resistor_SMD:R_1206_3216Metric_Pad1.30x1.75mm_HandSolder"
+		(property "Footprint" "Resistor_SMD:R_1206_3216Metric"
 			(at 110.49 151.892 90)
 			(effects
@@
 			)
 		)
-		(property "Footprint" "Resistor_SMD:R_1206_3216Metric_Pad1.30x1.75mm_HandSolder"
+		(property "Footprint" "Resistor_SMD:R_1206_3216Metric"
 			(at 95.25 259.842 90)
 			(effects
@@
 			)
 		)
-		(property "Footprint" "Resistor_SMD:R_1206_3216Metric_Pad1.30x1.75mm_HandSolder"
+		(property "Footprint" "Resistor_SMD:R_1206_3216Metric"
 			(at 95.25 214.122 90)
 			(effects
@@
 	)
 	(symbol
+		(lib_id "Connector_Generic:Conn_01x01")
+		(at 255.27 179.07 0)
+		(unit 1)
+		(exclude_from_sim no)
+		(in_bom yes)
+		(on_board yes)
+		(dnp no)
+		(fields_autoplaced yes)
+		(property "Reference" "J7"
+			(at 257.81 177.7999 0)
+			(effects
+				(font
+					(size 1.27 1.27)
+				)
+				(justify left)
+			)
+		)
+		(property "Value" "Conn_01x01"
+			(at 257.81 180.3399 0)
+			(effects
+				(font
+					(size 1.27 1.27)
+				)
+				(justify left)
+			)
+		)
+		(property "Footprint" "analog_NN:WireSolderPad_1.0mm"
+			(at 255.27 179.07 0)
+			(effects
+				(font
+					(size 1.27 1.27)
+				)
+				(hide yes)
+			)
+		)
+		(property "Datasheet" "~"
+			(at 255.27 179.07 0)
+			(effects
+				(font
+					(size 1.27 1.27)
+				)
+				(hide yes)
+			)
+		)
+		(property "Description" "Generic connector, single row, 01x01, script generated (kicad-library-utils/schlib/autogen/connector/)"
+			(at 255.27 179.07 0)
+			(effects
+				(font
+					(size 1.27 1.27)
+				)
+				(hide yes)
+			)
+		)
+		(pin "1"
+		)
+		(instances
+			(project ""
+				(path "/8de080c9-ac72-4350-b5d3-2d90d26f0ccc/34009bdb-0ff2-4f8c-b708-8950383cf335"
+					(reference "J7")
+					(unit 1)
+				)
+			)
+		)
+	)
+	(symbol
 		(lib_id "Device:C")
 		(at 166.37 222.25 180)
@@
 			)
 		)
-		(property "Footprint" "Capacitor_SMD:C_1206_3216Metric_Pad1.33x1.80mm_HandSolder"
+		(property "Footprint" "Capacitor_SMD:C_1206_3216Metric"
 			(at 165.4048 218.44 0)
 			(effects
@@
 			)
 		)
-		(property "Footprint" "Resistor_SMD:R_1206_3216Metric_Pad1.30x1.75mm_HandSolder"
+		(property "Footprint" "Resistor_SMD:R_1206_3216Metric"
 			(at 110.49 108.712 90)
 			(effects
@@
 			)
 		)
-		(property "Footprint" "Capacitor_SMD:C_1206_3216Metric_Pad1.33x1.80mm_HandSolder"
+		(property "Footprint" "Capacitor_SMD:C_1206_3216Metric"
 			(at 165.4048 90.17 0)
 			(effects
@@
 			)
 		)
-		(property "Footprint" "Capacitor_SMD:C_1206_3216Metric_Pad1.33x1.80mm_HandSolder"
+		(property "Footprint" "Capacitor_SMD:C_1206_3216Metric"
 			(at 187.6552 209.55 0)
 			(effects
@@
 			)
 		)
-		(property "Footprint" "Resistor_SMD:R_1206_3216Metric_Pad1.30x1.75mm_HandSolder"
+		(property "Footprint" "Resistor_SMD:R_1206_3216Metric"
 			(at 110.49 240.792 90)
 			(effects
@@
 			)
 		)
-		(property "Footprint" "Resistor_SMD:R_1206_3216Metric_Pad1.30x1.75mm_HandSolder"
+		(property "Footprint" "Resistor_SMD:R_1206_3216Metric"
 			(at 95.25 170.942 90)
 			(effects
@@
 			)
 		)
-		(property "Footprint" "Capacitor_SMD:C_1206_3216Metric_Pad1.33x1.80mm_HandSolder"
+		(property "Footprint" "Capacitor_SMD:C_1206_3216Metric"
 			(at 187.6552 271.78 0)
 			(effects
@@
 			)
 		)
-		(property "Footprint" "Capacitor_SMD:C_1206_3216Metric_Pad1.33x1.80mm_HandSolder"
+		(property "Footprint" "Capacitor_SMD:C_1206_3216Metric"
 			(at 187.6552 144.78 0)
 			(effects
@@
 			)
 		)
-		(property "Footprint" "Capacitor_SMD:C_1206_3216Metric_Pad1.33x1.80mm_HandSolder"
+		(property "Footprint" "Capacitor_SMD:C_1206_3216Metric"
 			(at 165.4048 280.67 0)
 			(effects
@@
 			)
 		)
-		(property "Footprint" "Resistor_SMD:R_1206_3216Metric_Pad1.30x1.75mm_HandSolder"
+		(property "Footprint" "Resistor_SMD:R_1206_3216Metric"
 			(at 95.25 127.762 90)
 			(effects
@@
 			)
 		)
-		(property "Footprint" "Capacitor_SMD:C_1206_3216Metric_Pad1.33x1.80mm_HandSolder"
+		(property "Footprint" "Capacitor_SMD:C_1206_3216Metric"
 			(at 165.4048 152.4 0)
 			(effects

Commit message: Fixed: v closed loop
Connections:
- net Vh1_forward renamed Vh1_back
- net Vh2_forward renamed Vh2_back
- net Vh3_forward renamed Vh3_back
- net Vh4_forward renamed Vh4_back
Changed lines of the file:
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@@
 		)
 	)
-	(global_label "Vh2_forward"
+	(global_label "Vh2_back"
 		(shape input)
 		(at 91.44 144.78 180)
@@
 		)
 		(property "Intersheetrefs" "${INTERSHEET_REFS}"
-			(at 76.9645 144.78 0)
+			(at 79.6254 144.78 0)
 			(effects
 				(font
@@
 		)
 	)
-	(global_label "Vh1_forward"
+	(global_label "Vh1_back"
 		(shape input)
 		(at 91.44 101.6 180)
@@
 		)
 		(property "Intersheetrefs" "${INTERSHEET_REFS}"
-			(at 76.9645 101.6 0)
-			(effects
-				(font
-					(size 1.27 1.27)
-				)
-				(justify right)
-				(hide yes)
-			)
-		)
-	)
-	(global_label "Vh4_forward"
+			(at 79.6254 101.6 0)
+			(effects
+				(font
+					(size 1.27 1.27)
+				)
+				(justify right)
+				(hide yes)
+			)
+		)
+	)
+	(global_label "Vh4_back"
 		(shape input)
 		(at 91.44 261.62 180)
@@
 		)
 		(property "Intersheetrefs" "${INTERSHEET_REFS}"
-			(at 76.9645 261.62 0)
+			(at 79.6254 261.62 0)
 			(effects
 				(font
@@
 		)
 	)
-	(global_label "Vh3_forward"
+	(global_label "Vh3_back"
 		(shape input)
 		(at 91.44 187.96 180)
@@
 		)
 		(property "Intersheetrefs" "${INTERSHEET_REFS}"
-			(at 76.9645 187.96 0)
+			(at 79.6254 187.96 0)
 			(effects
 				(font
@@
 		)
 	)
-	(global_label "Vh1_forward"
+	(global_label "Vh1_back"
 		(shape input)
 		(at 91.44 129.54 180)
@@
 		)
 		(property "Intersheetrefs" "${INTERSHEET_REFS}"
-			(at 76.9645 129.54 0)
+			(at 79.6254 129.54 0)
 			(effects
 				(font
@@
 		)
 	)
-	(global_label "Vh2_forward"
+	(global_label "Vh2_back"
 		(shape input)
 		(at 91.44 172.72 180)
@@
 		)
 		(property "Intersheetrefs" "${INTERSHEET_REFS}"
-			(at 76.9645 172.72 0)
+			(at 79.6254 172.72 0)
 			(effects
 				(font
@@
 		)
 	)
-	(global_label "Vh3_forward"
+	(global_label "Vh3_back"
 		(shape input)
 		(at 91.44 215.9 180)
@@
 		)
 		(property "Intersheetrefs" "${INTERSHEET_REFS}"
-			(at 76.9645 215.9 0)
+			(at 79.6254 215.9 0)
 			(effects
 				(font
@@
 		)
 	)
-	(global_label "Vh4_forward"
+	(global_label "Vh4_back"
 		(shape input)
 		(at 91.44 233.68 180)
@@
 		)
 		(property "Intersheetrefs" "${INTERSHEET_REFS}"
-			(at 76.9645 233.68 0)
-			(effects
-				(font
+			(at 79.6254 233.68 0)
+			(effects
+				(font
